File: Speccy2007_128K_Ljubitel.brd (EAGLE design)
At the start: 55.9 x 6.6 mm, 100 parts, among them X2 SCART-F, X5 ByteBlaster, X6 AVRISP

Commit message: .
Parts:
- added DD12: 74HCT04N, 74xx-eu:DIL14
- DD2: device altera_pga84:PGA-84 -> Speccy:PGA-84
- moved JP1 2.56 mm to (138.1, 32.4)
- moved R6P 2.56 mm to (133.0, 42.9)
- moved *R2 2.56 mm to (160.0, 17.1)
- moved C1Y 2.56 mm to (172.7, 29.5)
- moved C2Y 2.56 mm to (170.5, 31.1)
- moved C8P1 2.56 mm to (148.6, 30.5)
- moved C8P2 2.56 mm to (154.9, 30.5)
- moved DA1 2.56 mm to (147.0, 43.5)
- moved R8P 2.56 mm to (164.1, 31.8)
- moved R9P 2.56 mm to (132.7, 31.8)
- moved R9P1 2.56 mm to (152.4, 33.7)
- moved R9P2 2.56 mm to (158.4, 31.8)
- moved C9P 2.56 mm to (129.2, 30.5)
- moved C4P 2.56 mm to (149.5, 44.8)
- moved C5P 2.56 mm to (135.6, 42.9)
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Connections:
- new net VCC: DD12.14
- net GND: now also DD12.7
Routing:
- net WR: track 190.5 -> 236.4 mm, vias 4 -> 6
- net A0: track 106.8 -> 132.5 mm, vias 0 -> 2
- net ROM_A14: track 192.2 -> 185.8 mm
- net AVR_RST: track 0.00 -> 5.72 mm
- net +5V: track 441.8 -> 447.2 mm
- net WAIT_CPU: track 118.9 -> 122.1 mm
- net GND: track 626.8 -> 628.6 mm
- net VAGEN: track 177.1 -> 175.6 mm
- net D1: track 145.1 -> 143.7 mm
- net D5: track 166.1 -> 164.9 mm
- net INT: track 91.3 -> 90.2 mm
- net NMI: track 13.4 -> 14.5 mm
- net A12: track 224.1 -> 225.0 mm
- net D3: track 155.3 -> 154.5 mm
- net D4: track 152.3 -> 151.7 mm

Commit message: .
Parts:
- removed DD12: 74HCT04N, 74xx-eu:DIL14
- DD11: value 74HCT04N -> 74LS04N; device 74xx-eu:DIL14 -> Speccy:DIL14
- moved R7 1.59 mm to (156.2, 150.8)
- moved X5 0.63 mm to (157.5, 132.7)
Connections:
- removed net VCC: DD12.14
- net GND: no longer DD12.7
Routing:
- net BB: track 3.31 -> 4.86 mm
- net N$8: track 35.7 -> 37.0 mm
- net RD: track 261.3 -> 261.9 mm

Commit message: .
Parts:
- moved J1 4.80 mm to (173.7, 145.7)
- flipped RP1 to the top
- flipped RP2 to the top
Routing:
- net TDO: track 38.4 -> 41.0 mm
- net IOREQ: track 86.3 -> 84.0 mm
- net GND: track 628.6 -> 626.6 mm
- net +5V: track 447.7 -> 449.8 mm
- net D7: track 173.7 -> 171.9 mm
- net VAGEN: track 175.4 -> 176.6 mm

Commit message: .
Parts:
- added DD12: 74HC245N, Speccy:DIL20
- DD6: device memory-hitachi:DIL28-6 -> Speccy:DIL28+6
- R21: device rcl:0207/10 -> rcl:0207/12
- moved PS2KB 214.7 mm to (56.2, 20.6)
- moved R13 214.7 mm to (56.5, 38.1)
- moved R22 214.7 mm to (56.2, 32.4)
- moved R23 214.7 mm to (56.2, 34.9)
- moved *R2 142.8 mm to (259.7, 119.4), turned to 90 degrees
- moved X2 139.1 mm to (256.2, 104.8), turned to 90 degrees
- moved C9P 130.8 mm to (246.4, 88.6), turned to 0 degrees
- moved R9P 127.6 mm to (245.1, 92.1), turned to 270 degrees
- moved C1Y 126.8 mm to (247.3, 132.1), turned to 180 degrees
- moved C8P 125.9 mm to (246.4, 102.6), turned to 0 degrees
- moved C8P1 124.8 mm to (246.4, 108.0), turned to 0 degrees
- moved JP1 124.7 mm to (244.5, 97.5), turned to 180 degrees
- moved C2Y 124.1 mm to (245.7, 129.9), turned to 180 degrees
- moved C8P2 124.0 mm to (246.4, 114.3), turned to 0 degrees
- moved C6P 123.9 mm to (242.6, 92.7), turned to 270 degrees
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Connections:
- new net VCC: DD12.20
- net GND: now also DD12.10, DD6.P$14
- net VA1: now also DD6.P$6
- net VA11: now also DD6.P$7
- net VA12: now also DD6.P$8
- net VA13: now also DD6.P$9
- net VA14: now also DD6.P$10
- net VA2: now also DD6.P$5
- net VA3: now also DD6.P$4
- net VA4: now also DD6.P$3
- net VA5: now also DD6.P$1
- net VA6: now also DD6.P$2
- net VD1: now also DD6.P$13
- net VD5: now also DD6.P$11
- net VD7: now also DD6.P$12
Routing:
- net N$9: track 49.9 -> 28.1 mm
- net +5V: track 449.8 -> 460.7 mm
- net WR: track 236.4 -> 244.9 mm
- net D7: track 171.9 -> 179.9 mm
- net A15: track 164.1 -> 157.2 mm
- net TDO: track 41.0 -> 47.6 mm
- net TCK: track 33.0 -> 39.1 mm
- net CLK_CPU: track 126.8 -> 121.3 mm
- net RA15: track 124.3 -> 129.7 mm
- net WAIT_CPU: track 122.1 -> 116.7 mm
- net RD: track 261.9 -> 267.1 mm
- net RA14: track 134.3 -> 139.4 mm
- net ROM_A14: track 185.8 -> 190.8 mm
- net G: track 5.13 -> 9.68 mm
- net ROM_A15: track 100.9 -> 96.6 mm
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Other:
- board size 55.9 x 6.6 mm -> 6.6 x 55.9 mm

Commit message: .
Parts:
- removed DD12: 74HC245N, Speccy:DIL20
- removed RP1, RP2: (no value), con-lsta:FE07
- added R1: (no value), rcl:M1206
- R21: device rcl:0207/12 -> Speccy:0207/10
- moved R13 162.8 mm to (185.4, 137.5)
- moved *R2 143.8 mm to (161.9, 14.0), turned to 180 degrees
- moved X2 139.6 mm to (147.3, 17.5), turned to 0 degrees
- moved C9P 130.5 mm to (131.1, 27.3), turned to 270 degrees
- moved C1Y 128.3 mm to (174.6, 26.4), turned to 270 degrees
- moved R9P 127.4 mm to (134.6, 28.6), turned to 0 degrees
- moved C8P 126.2 mm to (145.1, 27.3), turned to 270 degrees
- moved C2Y 125.6 mm to (172.4, 27.9), turned to 270 degrees
- moved C8P1 125.3 mm to (150.5, 27.3), turned to 270 degrees
- moved C8P2 124.8 mm to (156.8, 27.3), turned to 270 degrees
- moved JP1 124.8 mm to (140.0, 29.2), turned to 90 degrees
- moved C6P 123.7 mm to (135.3, 31.1), turned to 180 degrees
- moved R8P 123.5 mm to (166.1, 28.6), turned to 0 degrees
- moved R9P2 123.1 mm to (160.3, 28.6), turned to 0 degrees
- moved R9P1 120.5 mm to (154.3, 30.5), turned to 270 degrees
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Connections:
- removed net VCC: DD12.20
- net GND: no longer DD12.10
Routing:
- net A8: track 153.3 -> 233.8 mm, vias 0 -> 1
- net A9: track 157.3 -> 226.7 mm, vias 1 -> 2
- net ROM_A15: track 96.6 -> 110.0 mm
- net AVR_TRDOS: track 30.2 -> 19.1 mm
- net D7: track 179.9 -> 190.4 mm, vias 2 -> 4
- net GND: track 629.0 -> 638.7 mm
- net CLK: track 25.8 -> 17.3 mm
- net WAIT_CPU: track 116.7 -> 108.6 mm
- net AVR_NOINT: track 32.7 -> 26.8 mm
- net WR: track 244.9 -> 239.0 mm
- net AY_BDIR: track 27.9 -> 22.2 mm
- net A5: track 149.4 -> 153.2 mm
- net A10: track 206.8 -> 203.1 mm
- net ROM_A14: track 190.8 -> 187.2 mm
- net A3: track 140.6 -> 143.7 mm
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Other:
- board size 6.6 x 55.9 mm -> 55.9 x 6.6 mm

Commit message: .
Parts:
- moved R21 0.32 mm to (82.4, 95.2)
Routing:
- net ROM_A15: track 110.0 -> 174.6 mm, vias 0 -> 3
- net ROM_CS: track 133.3 -> 139.3 mm
- net CLK_CPU: track 122.0 -> 125.9 mm
- net MREQ: track 84.3 -> 80.9 mm
- net INT: track 91.4 -> 94.7 mm
- net A10: track 203.1 -> 206.0 mm
- net WR: track 239.0 -> 241.6 mm
- net A15: track 158.8 -> 160.8 mm
- net RD: track 268.9 -> 270.4 mm
- net WAIT_CPU: track 108.6 -> 110.1 mm
- net D6: track 184.8 -> 185.8 mm
- net M1: track 115.4 -> 114.8 mm
- net D7: track 190.4 -> 189.8 mm

Commit message: .
Parts:
- moved C8 173.1 mm to (62.2, 15.2)
- moved C9 173.1 mm to (59.1, 22.9)
- moved J1 173.1 mm to (58.1, 16.8)
- moved R11 173.1 mm to (66.7, 10.5)
- moved R12 173.1 mm to (61.6, 6.99)
- moved R13 173.1 mm to (69.8, 8.57)
- moved R14 173.1 mm to (58.4, 11.7)
- moved R15 173.1 mm to (54.0, 10.2)
- moved R16 173.1 mm to (54.0, 14.0)
- moved R17 173.1 mm to (64.8, 21.3)
- moved R18 173.1 mm to (67.3, 21.3)
- moved VT1 173.1 mm to (65.4, 26.4)
- moved X6 173.1 mm to (68.6, 15.2)
- moved *R2 164.4 mm to (292.4, 114.0), turned to 90 degrees
- moved X2 163.6 mm to (288.9, 99.4), turned to 90 degrees
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Routing:
- net A14: track 30.6 -> 133.3 mm, vias 0 -> 1
- net AVR_NOINT: track 26.8 -> 106.2 mm, vias 2 -> 1
- net AVR_WAIT: track 4.79 -> 82.0 mm, vias 0 -> 2
- net AVR_INT: track 13.2 -> 85.5 mm
- net SPEAKER: track 42.4 -> 113.5 mm
- net TAPE_IN: track 23.3 -> 88.2 mm
- net CLK: track 17.3 -> 74.0 mm, vias 1 -> 3
- net AVR_PROM: track 26.3 -> 81.7 mm, vias 1 -> 3
- net AVR_TRDOS: track 19.1 -> 72.3 mm, vias 0 -> 3
- net D7: track 189.8 -> 237.4 mm
- net D6: track 185.8 -> 231.3 mm
- net D4: track 153.8 -> 196.9 mm
- net D3: track 154.6 -> 194.9 mm
- net D2: track 123.5 -> 163.0 mm
- net D5: track 163.2 -> 202.2 mm
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Other:
- board size 55.9 x 6.6 mm -> 6.6 x 55.9 mm

Commit message: .
Parts:
- moved C9 173.8 mm to (175.3, 152.1)
- moved J1 173.8 mm to (174.3, 146.1)
- moved C8 173.8 mm to (178.4, 144.5)
- moved R12 173.8 mm to (177.8, 136.2)
- moved R13 173.8 mm to (186.1, 137.8)
- moved R15 173.8 mm to (170.2, 139.4)
- moved R16 173.8 mm to (170.2, 143.2)
- moved VT1 173.8 mm to (181.6, 155.6)
- moved R11 173.8 mm to (182.9, 139.7)
- moved R14 173.8 mm to (174.6, 141.0)
- moved R17 173.8 mm to (181.0, 150.5)
- moved R18 173.8 mm to (183.5, 150.5)
- moved X6 162.1 mm to (170.5, 141.3)
- moved C1Y 152.9 mm to (134.3, 80.3), turned to 270 degrees
- moved C2Y 144.9 mm to (140.3, 80.6)
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Routing:
- net KCLK: track 0.00 -> 85.1 mm
- net KDAT: track 0.00 -> 79.3 mm
- net RST_CPU: track 115.2 -> 135.0 mm
- net A12: track 224.4 -> 242.6 mm
- net SPEAKER: track 113.5 -> 99.4 mm
- net +5V: track 458.7 -> 472.7 mm
- net GND: track 638.0 -> 624.5 mm
- net AY_CLK: track 51.3 -> 63.0 mm
- net D0: track 176.6 -> 167.9 mm
- net D1: track 182.2 -> 174.3 mm
- net D2: track 163.0 -> 156.5 mm
- net AVR_TRDOS: track 72.3 -> 78.6 mm, vias 3 -> 2
- net D4: track 196.9 -> 191.1 mm
- net AY_BC: track 36.5 -> 42.0 mm
- net AY_BDIR: track 50.3 -> 55.8 mm
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Other:
- board size 6.6 x 55.9 mm -> 168.9 x 114.6 mm
