File: Speccy2007_128K_Ljubitel.brd (EAGLE design)
At the start: 168.6 x 112.4 mm, 114 parts, among them X1 5V, X2 SCART-F, X3 PS/2 KB, X4 SD Card, X5 ByteBlaster, X6 AVRISP

Commit message: .
Parts:
- CRL: device rcl:C1206 -> rcl:C0805
- moved R4 1.80 mm to (55.9, 12.1), turned to 270 degrees
- moved R34 1.77 mm to (12.4, 47.0), turned to 90 degrees
- moved Z1 0.63 mm to (14.9, 43.7)
- moved Z2 0.32 mm to (33.7, 63.3)
Routing:
- net GND: track 1193.6 -> 1201.6 mm, vias 6 -> 7
- net +5V: track 759.9 -> 766.3 mm
- net ROM_A15: track 172.6 -> 175.7 mm
- net A15: track 155.8 -> 157.9 mm
- net BG: track 15.8 -> 17.7 mm
- net N$12: track 5.21 -> 7.11 mm
- net WR: track 234.3 -> 236.0 mm
- net VD6: track 77.9 -> 79.7 mm
- net VD4: track 85.7 -> 87.5 mm
- net RD: track 259.6 -> 261.3 mm
- net ROM_A14: track 182.5 -> 184.2 mm
- net BR: track 5.97 -> 7.55 mm
- net M1: track 112.6 -> 114.0 mm
- net IOREQ: track 77.5 -> 78.9 mm
- net AVR_PROM: track 85.9 -> 87.4 mm
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
Commit message: .
Routing:
- net SDC: track 111.1 -> 112.5 mm
- net MOSI: track 127.0 -> 128.2 mm
- net MISO: track 130.2 -> 131.2 mm
Changed lines of the file:
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@@
 <wire x1="129.8575" y1="86.83625" x2="136.525" y2="84.29625" width="0.3048" layer="16"/>
 <wire x1="136.525" y1="84.29625" x2="138.1125" y2="84.29625" width="0.3048" layer="16"/>
-<wire x1="133.6675" y1="31.90875" x2="133.6675" y2="24.93625" width="0.4064" layer="1"/>
-<wire x1="133.6675" y1="24.93625" x2="131.7625" y2="23.03125" width="0.4064" layer="1"/>
+<wire x1="133.50875" y1="32.0675" x2="133.50875" y2="24.7775" width="0.4064" layer="1"/>
+<wire x1="133.50875" y1="24.7775" x2="131.7625" y2="23.03125" width="0.4064" layer="1"/>
 <wire x1="131.7625" y1="23.03125" x2="130.055" y2="23.03125" width="0.4064" layer="1"/>
 <wire x1="140.0175" y1="59.53125" x2="140.0175" y2="56.67375" width="0.3048" layer="1"/>
 <wire x1="131.445" y1="46.19625" x2="132.3975" y2="45.24375" width="0.4064" layer="1"/>
 <wire x1="132.3975" y1="45.24375" x2="132.3975" y2="33.17875" width="0.4064" layer="1"/>
-<wire x1="132.3975" y1="33.17875" x2="133.6675" y2="31.90875" width="0.4064" layer="1"/>
+<wire x1="132.3975" y1="33.17875" x2="133.50875" y2="32.0675" width="0.4064" layer="1"/>
 <wire x1="131.445" y1="46.19625" x2="131.445" y2="51.59375" width="0.4064" layer="1"/>
 <wire x1="131.445" y1="51.59375" x2="133.985" y2="54.13375" width="0.4064" layer="1"/>
@@
 <wire x1="100.965" y1="81.75625" x2="100.33" y2="82.39125" width="0.4064" layer="1"/>
 <wire x1="100.33" y1="82.39125" x2="99.695" y2="83.66125" width="0.4064" layer="1"/>
-<wire x1="89.2175" y1="60.16625" x2="88.5825" y2="59.53125" width="0.4064" layer="1"/>
-<wire x1="88.5825" y1="59.53125" x2="84.7725" y2="59.53125" width="0.4064" layer="1"/>
-<wire x1="84.7725" y1="59.53125" x2="82.8675" y2="61.43625" width="0.4064" layer="1"/>
-<wire x1="82.8675" y1="61.43625" x2="82.8675" y2="63.34125" width="0.4064" layer="1"/>
+<wire x1="89.2175" y1="60.16625" x2="88.265" y2="59.21375" width="0.4064" layer="1"/>
+<wire x1="88.265" y1="59.21375" x2="84.7725" y2="59.21375" width="0.4064" layer="1"/>
+<wire x1="84.7725" y1="59.21375" x2="82.8675" y2="61.11875" width="0.4064" layer="1"/>
+<wire x1="82.8675" y1="61.11875" x2="82.8675" y2="63.34125" width="0.4064" layer="1"/>
 <wire x1="82.8675" y1="63.34125" x2="78.105" y2="68.10375" width="0.4064" layer="1"/>
 <wire x1="78.105" y1="68.10375" x2="47.3075" y2="68.10375" width="0.4064" layer="1"/>
@@
 <wire x1="101.9175" y1="71.59625" x2="99.695" y2="71.59625" width="0.4064" layer="1"/>
 <wire x1="99.695" y1="71.59625" x2="96.52" y2="68.42125" width="0.4064" layer="1"/>
-<wire x1="96.52" y1="68.42125" x2="96.52" y2="56.03875" width="0.4064" layer="1"/>
-<wire x1="96.52" y1="56.03875" x2="94.9325" y2="54.45125" width="0.4064" layer="1"/>
-<wire x1="94.9325" y1="54.45125" x2="82.8675" y2="54.45125" width="0.4064" layer="1"/>
-<wire x1="82.8675" y1="54.45125" x2="77.7875" y2="59.53125" width="0.4064" layer="1"/>
-<wire x1="77.7875" y1="59.53125" x2="77.7875" y2="61.11875" width="0.4064" layer="1"/>
+<wire x1="96.52" y1="68.42125" x2="96.52" y2="55.08625" width="0.4064" layer="1"/>
+<wire x1="96.52" y1="55.08625" x2="95.5675" y2="54.13375" width="0.4064" layer="1"/>
+<wire x1="95.5675" y1="54.13375" x2="82.2325" y2="54.13375" width="0.4064" layer="1"/>
+<wire x1="82.2325" y1="54.13375" x2="77.7875" y2="58.57875" width="0.4064" layer="1"/>
+<wire x1="77.7875" y1="58.57875" x2="77.7875" y2="61.11875" width="0.4064" layer="1"/>
 <wire x1="77.7875" y1="61.11875" x2="74.93" y2="63.97625" width="0.4064" layer="1"/>
 <wire x1="74.93" y1="63.97625" x2="49.53" y2="63.97625" width="0.4064" layer="1"/>
@@
 <wire x1="101.9175" y1="74.13625" x2="100.33" y2="74.13625" width="0.4064" layer="1"/>
 <wire x1="100.33" y1="74.13625" x2="95.25" y2="69.05625" width="0.4064" layer="1"/>
-<wire x1="95.25" y1="69.05625" x2="95.25" y2="57.30875" width="0.4064" layer="1"/>
-<wire x1="95.25" y1="57.30875" x2="93.6625" y2="55.72125" width="0.4064" layer="1"/>
-<wire x1="93.6625" y1="55.72125" x2="83.185" y2="55.72125" width="0.4064" layer="1"/>
-<wire x1="83.185" y1="55.72125" x2="79.0575" y2="59.84875" width="0.4064" layer="1"/>
-<wire x1="79.0575" y1="59.84875" x2="79.0575" y2="61.75375" width="0.4064" layer="1"/>
+<wire x1="95.25" y1="69.05625" x2="95.25" y2="56.35625" width="0.4064" layer="1"/>
+<wire x1="95.25" y1="56.35625" x2="94.2975" y2="55.40375" width="0.4064" layer="1"/>
+<wire x1="94.2975" y1="55.40375" x2="82.8675" y2="55.40375" width="0.4064" layer="1"/>
+<wire x1="82.8675" y1="55.40375" x2="79.0575" y2="59.21375" width="0.4064" layer="1"/>
+<wire x1="79.0575" y1="59.21375" x2="79.0575" y2="61.75375" width="0.4064" layer="1"/>
 <wire x1="79.0575" y1="61.75375" x2="75.565" y2="65.24625" width="0.4064" layer="1"/>
 <wire x1="75.565" y1="65.24625" x2="49.2125" y2="65.24625" width="0.4064" layer="1"/>
@@
 <wire x1="101.9175" y1="76.67625" x2="100.6475" y2="76.67625" width="0.4064" layer="1"/>
 <wire x1="100.6475" y1="76.67625" x2="93.6625" y2="69.69125" width="0.4064" layer="1"/>
-<wire x1="93.6625" y1="69.69125" x2="93.6625" y2="58.26125" width="0.4064" layer="1"/>
+<wire x1="93.6625" y1="69.69125" x2="93.6625" y2="57.62625" width="0.4064" layer="1"/>
 <wire x1="76.5175" y1="66.19875" x2="80.3275" y2="62.38875" width="0.4064" layer="1"/>
-<wire x1="80.3275" y1="62.38875" x2="80.3275" y2="60.48375" width="0.4064" layer="1"/>
-<wire x1="80.3275" y1="60.48375" x2="83.82" y2="56.99125" width="0.4064" layer="1"/>
-<wire x1="83.82" y1="56.99125" x2="92.3925" y2="56.99125" width="0.4064" layer="1"/>
-<wire x1="92.3925" y1="56.99125" x2="93.6625" y2="58.26125" width="0.4064" layer="1"/>
+<wire x1="80.3275" y1="62.38875" x2="80.3275" y2="59.84875" width="0.4064" layer="1"/>
+<wire x1="80.3275" y1="59.84875" x2="83.5025" y2="56.67375" width="0.4064" layer="1"/>
+<wire x1="83.5025" y1="56.67375" x2="92.71" y2="56.67375" width="0.4064" layer="1"/>
+<wire x1="92.71" y1="56.67375" x2="93.6625" y2="57.62625" width="0.4064" layer="1"/>
 <wire x1="76.5175" y1="66.19875" x2="48.5775" y2="66.19875" width="0.4064" layer="1"/>
 <via x="19.84375" y="37.465" extent="1-16" drill="0.8" diameter="2.1844"/>
@@
 <wire x1="97.155" y1="77.94625" x2="90.17" y2="70.96125" width="0.4064" layer="1"/>
 <wire x1="90.17" y1="70.96125" x2="90.17" y2="59.53125" width="0.4064" layer="1"/>
-<wire x1="90.17" y1="59.53125" x2="88.9" y2="58.26125" width="0.4064" layer="1"/>
-<wire x1="88.9" y1="58.26125" x2="84.1375" y2="58.26125" width="0.4064" layer="1"/>
-<wire x1="84.1375" y1="58.26125" x2="81.5975" y2="60.80125" width="0.4064" layer="1"/>
-<wire x1="81.5975" y1="60.80125" x2="81.5975" y2="62.70625" width="0.4064" layer="1"/>
+<wire x1="90.17" y1="59.53125" x2="88.5825" y2="57.94375" width="0.4064" layer="1"/>
+<wire x1="88.5825" y1="57.94375" x2="84.1375" y2="57.94375" width="0.4064" layer="1"/>
+<wire x1="84.1375" y1="57.94375" x2="81.5975" y2="60.48375" width="0.4064" layer="1"/>
+<wire x1="81.5975" y1="60.48375" x2="81.5975" y2="62.70625" width="0.4064" layer="1"/>
 <wire x1="81.5975" y1="62.70625" x2="77.1525" y2="67.15125" width="0.4064" layer="1"/>
 <wire x1="77.1525" y1="67.15125" x2="47.9425" y2="67.15125" width="0.4064" layer="1"/>

Commit message: .
Parts:
- R19: device rcl:M1206 -> rcl:M0805
- moved R19 1.27 mm to (105.4, 83.0)
Routing:
- net AVR_RST: track 129.0 -> 127.9 mm
- net +5V: track 766.3 -> 767.4 mm

Commit message: .
Routing:
- net GND: track 1201.6 -> 1210.7 mm, vias 7 -> 9
- net IOREQ: track 78.9 -> 81.7 mm
- net ROM_A15: track 175.7 -> 178.3 mm
- net ROM_A14: track 184.2 -> 186.7 mm
- net A15: track 157.9 -> 159.6 mm
- net MREQ: track 78.4 -> 79.8 mm
- net VA13: track 29.5 -> 30.9 mm
- net WAIT_CPU: track 93.0 -> 94.1 mm
- net VD3: track 89.4 -> 90.5 mm

Commit message: .
Routing:
- net +5V: track 767.4 -> 848.6 mm
- net A9: track 227.7 -> 260.2 mm
- net A13: track 227.4 -> 214.0 mm
- net AVR_NOINT: track 105.8 -> 101.3 mm
- net ROM_A15: track 178.3 -> 173.9 mm
- net A11: track 283.7 -> 282.3 mm
- net RD: track 261.3 -> 262.3 mm

Commit message: .
Parts:
- R26: device rcl:R0805 -> rcl:R1206
- moved C2P 8.47 mm to (16.5, 14.8)
- moved C1P 2.51 mm to (6.51, 23.8), turned to 90 degrees
- moved R26 1.92 mm to (11.3, 23.8), turned to 180 degrees
- moved C3P 1.91 mm to (6.99, 17.6)
- moved R25 1.35 mm to (9.21, 37.3)
- moved HL1 0.63 mm to (12.1, 33.8)
- moved HL2 0.63 mm to (12.1, 28.7)
Routing:
- net GND: track 1210.7 -> 1220.5 mm
- net N$35: track 77.3 -> 87.1 mm
- net N$14: track 37.1 -> 28.0 mm
- net +3V3: track 61.3 -> 64.7 mm
- net N$41: track 1.81 -> 4.79 mm
- net N$47: track 63.2 -> 60.5 mm
- net N$11: track 53.0 -> 55.7 mm
- net N$46: track 69.2 -> 71.3 mm
- net N$13: track 46.8 -> 44.9 mm
- net N$22: track 117.4 -> 119.0 mm
- net SPEAKER: track 213.9 -> 215.3 mm
- net N$39: track 2.39 -> 3.48 mm
- net N$16: track 43.3 -> 42.8 mm

Commit message: .
Parts:
- added R1, R28, R29: 1k, rcl:R0805
Connections:
- new net N$23: DD10.1, R1.1
- new net N$24: DD5.1, DD5.2, DD5.3, R28.1
- new net N$42: DD4.1, R29.1
- net +5V: now also R1.2, R28.2, R29.2; no longer DD10.1, DD4.1, DD5.1, DD5.2, DD5.3
Routing:
- net VAGEN: track 166.5 -> 183.3 mm, vias 2 -> 3
- net N$24: track 0.00 -> 7.82 mm
- net RAM_CS: track 159.8 -> 154.3 mm
- net N$42: track 0.00 -> 2.87 mm
- net N$23: track 0.00 -> 2.55 mm
Other:
- board text added: "Speccy2007 DIP 128KB Y"
- board text removed: "Speccy2007 128KB Y"

Commit message: .
Parts:
- added C1: (no value), Speccy:E3,5-8
- moved CX1 8.80 mm to (72.4, 94.0), turned to 270 degrees
Connections:
- net +5V: now also C1.+
- net GND: now also C1.-
Routing:
- net +5V: track 848.9 -> 860.7 mm
- net GND: track 1220.5 -> 1230.1 mm
- net N$58: track 0.00 -> 3.18 mm
- net N$56: track 0.00 -> 3.18 mm
- net N$55: track 0.00 -> 3.18 mm
- net N$54: track 0.00 -> 3.18 mm
- net N$60: track 0.00 -> 3.18 mm
- net N$59: track 0.00 -> 3.18 mm
- net N$51: track 0.00 -> 3.17 mm
- net N$48: track 0.00 -> 3.17 mm
Changed lines of the file:
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@@
 </element>
 <element name="C9P" library="Speccy" package="E2,5-5" value="220mf" x="65.7225" y="99.21875" smashed="yes" rot="R270">
-<attribute name="NAME" x="64.643" y="95.09125" size="1.27" layer="25" ratio="10"/>
-<attribute name="VALUE" x="64.643" y="93.31325" size="1.27" layer="27" ratio="10"/>
+<attribute name="NAME" x="68.453" y="100.17125" size="1.27" layer="25" ratio="10"/>
+<attribute name="VALUE" x="68.7705" y="98.39325" size="1.27" layer="27" ratio="10"/>
 </element>
 <element name="R5P" library="rcl" package="M1206" value="16k*" x="15.5575" y="74.77125" smashed="yes" rot="MR180">
@@
 <attribute name="VALUE" x="73.3425" y="40.3225" size="1.27" layer="28" rot="MR0"/>
 </element>
-<element name="CX1" library="rcl" package="C0805" value="100n" x="76.2" y="101.9175" rot="MR0"/>
+<element name="CX1" library="rcl" package="C0805" value="100n" x="72.39" y="93.98" rot="MR270"/>
 <element name="R1" library="rcl" package="R0805" value="1k" x="156.5275" y="54.61" smashed="yes" rot="MR270">
 <attribute name="NAME" x="158.90875" y="56.67375" size="1.27" layer="26" rot="MR180"/>
@@
 <attribute name="VALUE" x="112.395" y="2.69875" size="1.27" layer="28" rot="MR0"/>
 </element>
+<element name="C1" library="Speccy" package="E3,5-8" value="" x="70.1675" y="93.6625" rot="R270"/>
 </elements>
 <signals>
@@
 <wire x1="80.01" y1="107.79125" x2="77.26" y2="105.29125" width="0.8128" layer="16"/>
 <wire x1="80.01" y1="88.10625" x2="77.1525" y2="88.10625" width="0.8128" layer="1"/>
-<wire x1="73.3425" y1="100.33" x2="73.3425" y2="93.50375" width="0.8128" layer="16"/>
 <wire x1="39.6875" y1="55.72125" x2="39.6875" y2="56.67375" width="0.4064" layer="1"/>
 <wire x1="39.6875" y1="56.67375" x2="40.64" y2="57.62625" width="0.4064" layer="1"/>
@@
 <wire x1="63.02375" y1="20.955" x2="62.23" y2="19.20875" width="0.3048" layer="1"/>
 <contactref element="CX1" pad="2"/>
-<wire x1="75.25" y1="101.9175" x2="73.3425" y2="100.33" width="0.8128" layer="16"/>
 <wire x1="77.26" y1="105.29125" x2="75.25" y2="103.70375" width="0.8128" layer="16"/>
-<wire x1="75.25" y1="103.70375" x2="75.25" y2="101.9175" width="0.8128" layer="16"/>
-<wire x1="77.1525" y1="88.10625" x2="77.1525" y2="89.69375" width="0.8128" layer="16"/>
-<wire x1="77.1525" y1="89.69375" x2="73.3425" y2="93.50375" width="0.8128" layer="16"/>
+<wire x1="77.1525" y1="88.10625" x2="77.1525" y2="90.64625" width="0.8128" layer="16"/>
 <wire x1="62.23" y1="19.20875" x2="62.23" y2="20.32" width="1.016" layer="16"/>
 <wire x1="62.23" y1="20.32" x2="61.43625" y2="20.6375" width="0.4064" layer="16"/>
@@
 <wire x1="11.27125" y1="24.92375" x2="12.22375" y2="25.87625" width="0.3048" layer="1"/>
 <wire x1="12.22375" y1="25.87625" x2="14.176375" y2="25.87625" width="0.3048" layer="1"/>
+<contactref element="C1" pad="-"/>
+<wire x1="77.1525" y1="90.64625" x2="75.91425" y2="91.8845" width="0.8128" layer="16"/>
+<wire x1="75.91425" y1="91.8845" x2="72.39" y2="91.8845" width="0.8128" layer="16"/>
+<wire x1="72.39" y1="91.8845" x2="70.1675" y2="91.8845" width="0.8128" layer="16"/>
+<wire x1="75.25" y1="103.70375" x2="67.6275" y2="96.08125" width="0.8128" layer="16"/>
+<wire x1="67.6275" y1="96.08125" x2="67.6275" y2="93.6625" width="0.8128" layer="16"/>
+<wire x1="67.6275" y1="93.6625" x2="69.4055" y2="91.8845" width="0.8128" layer="16"/>
+<wire x1="69.4055" y1="91.8845" x2="70.1675" y2="91.8845" width="0.8128" layer="16"/>
+<wire x1="72.39" y1="93.03" x2="72.39" y2="91.8845" width="0.8128" layer="16"/>
 <wire x1="7.46125" y1="42.545" x2="9.2075" y2="38.25625" width="0" layer="19" extent="1-1"/>
 </signal>
@@
 <wire x1="57.15" y1="13.335" x2="63.1825" y2="13.335" width="0.4064" layer="1"/>
 <contactref element="CX1" pad="1"/>
-<wire x1="77.15" y1="101.9175" x2="80.01" y2="102.79125" width="0.8128" layer="16"/>
 <wire x1="40.9575" y1="35.71875" x2="40.9575" y2="43.33875" width="0.4064" layer="16"/>
 <wire x1="62.23" y1="47.14875" x2="62.23" y2="48.895" width="1.016" layer="1"/>
@@
 <wire x1="122.435" y1="3.6125" x2="122.555" y2="3.4925" width="0.6096" layer="16"/>
 <wire x1="125.26875" y1="5.25125" x2="122.435" y2="5.25125" width="0.6096" layer="16"/>
+<contactref element="C1" pad="+"/>
+<wire x1="70.1675" y1="95.4405" x2="70.866" y2="96.139" width="0.8128" layer="16"/>
+<wire x1="70.866" y1="96.139" x2="77.51825" y2="102.79125" width="0.8128" layer="16"/>
+<wire x1="77.51825" y1="102.79125" x2="80.01" y2="102.79125" width="0.8128" layer="16"/>
+<wire x1="72.39" y1="94.93" x2="70.866" y2="96.1365" width="0.8128" layer="16"/>
+<wire x1="70.866" y1="96.1365" x2="70.866" y2="96.139" width="0.8128" layer="16"/>
 <wire x1="74.6125" y1="42.5425" x2="74.295" y2="33.3375" width="0" layer="19" extent="16-16"/>
 <wire x1="40.9575" y1="43.33875" x2="52.07" y2="44.60875" width="0" layer="19" extent="16-16"/>
@@
 <wire x1="72.0725" y1="83.34625" x2="73.03" y2="83.34625" width="0.8128" layer="16"/>
 <wire x1="73.03" y1="83.34625" x2="74.4605" y2="83.97875" width="0.8128" layer="16"/>
-<wire x1="68.2625" y1="89.37625" x2="68.2625" y2="90.96375" width="0.4064" layer="16"/>
+<wire x1="68.2625" y1="89.37625" x2="68.2625" y2="90.64625" width="0.4064" layer="16"/>
 <wire x1="56.1975" y1="91.28125" x2="58.7375" y2="94.45625" width="0.4064" layer="16"/>
-<wire x1="68.2625" y1="90.96375" x2="64.77" y2="94.45625" width="0.4064" layer="16"/>
-<wire x1="64.77" y1="94.45625" x2="58.7375" y2="94.45625" width="0.4064" layer="16"/>
+<wire x1="68.2625" y1="90.64625" x2="64.4525" y2="94.45625" width="0.4064" layer="16"/>
+<wire x1="64.4525" y1="94.45625" x2="58.7375" y2="94.45625" width="0.4064" layer="16"/>
 <wire x1="56.1975" y1="91.28125" x2="32.385" y2="91.28125" width="0.4064" layer="16"/>
 <wire x1="32.385" y1="91.28125" x2="31.115" y2="92.55125" width="0.4064" layer="16"/>
@@
 <signal name="N$26">
 <via x="165.4175" y="88.10625" extent="1-16" drill="3.2" diameter="5"/>
+<via x="6.985" y="107.47375" extent="1-16" drill="3.2" diameter="5"/>
 </signal>
 <signal name="V_OUT">
@@
 <wire x1="115.57" y1="5.23875" x2="115.58" y2="5.24875" width="0.6096" layer="16"/>
 </signal>
+<signal name="N$48">
+<wire x1="1.905" y1="1.5875" x2="1.905" y2="3.175" width="0.6096" layer="16"/>
+<wire x1="1.905" y1="1.5875" x2="3.4925" y2="1.5875" width="0.6096" layer="16"/>
+</signal>
+<signal name="N$51">
+<wire x1="1.905" y1="3.175" x2="1.905" y2="1.5875" width="0.6096" layer="1"/>
+<wire x1="1.905" y1="1.5875" x2="3.4925" y2="1.5875" width="0.6096" layer="1"/>
+</signal>
+<signal name="N$54">
+<wire x1="1.905" y1="113.9825" x2="1.905" y2="112.395" width="0.6096" layer="1"/>
+<wire x1="1.905" y1="113.9825" x2="3.4925" y2="113.9825" width="0.6096" layer="1"/>
+</signal>
+<signal name="N$55">
+<wire x1="1.905" y1="112.395" x2="1.905" y2="113.9825" width="0.6096" layer="16"/>
+<wire x1="1.905" y1="113.9825" x2="3.4925" y2="113.9825" width="0.6096" layer="16"/>
+</signal>
+<signal name="N$56">
+<wire x1="170.4975" y1="113.9825" x2="168.91" y2="113.9825" width="0.6096" layer="16"/>
+<wire x1="170.4975" y1="113.9825" x2="170.4975" y2="112.395" width="0.6096" layer="16"/>
+</signal>
+<signal name="N$58">
+<wire x1="168.91" y1="113.9825" x2="170.4975" y2="113.9825" width="0.6096" layer="1"/>
+<wire x1="170.4975" y1="113.9825" x2="170.4975" y2="112.395" width="0.6096" layer="1"/>
+</signal>
+<signal name="N$59">
+<wire x1="170.4975" y1="1.5875" x2="168.91" y2="1.5875" width="0.6096" layer="16"/>
+<wire x1="170.4975" y1="1.5875" x2="170.4975" y2="3.175" width="0.6096" layer="16"/>
+</signal>
+<signal name="N$60">
+<wire x1="168.91" y1="1.5875" x2="170.4975" y2="1.5875" width="0.6096" layer="1"/>
+<wire x1="170.4975" y1="1.5875" x2="170.4975" y2="3.175" width="0.6096" layer="1"/>
+</signal>
 </signals>
