File: Speccy2007_128K_Ljubitel.brd (EAGLE design)
At the start: 168.6 x 112.4 mm, 118 parts, among them X1 5V, X2 SCART-F, X3 PS/2 KB, X4 SD Card, X5 ByteBlaster, X6 AVRISP

Commit message: .....
Parts:
- DA1: value CXA1645 -> CXA1645P
- DD11: value 74LS04N -> К555ЛН1
- DD12: value 74LS74O -> К155ТМ2
- DD2: value EPM7128-J84 -> EPM7128SLC84-15
- R2: value (none) -> 0
- R6P: device rcl:R1206 -> rcl:R0805
Routing:
- net GND: track 1230.8 -> 1243.6 mm, vias 9 -> 11
Changed lines of the file:
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@@
 <layer number="23" name="tOrigins" color="15" fill="1" visible="yes" active="yes"/>
 <layer number="24" name="bOrigins" color="15" fill="1" visible="yes" active="yes"/>
-<layer number="25" name="tNames" color="7" fill="1" visible="no" active="yes"/>
+<layer number="25" name="tNames" color="7" fill="1" visible="yes" active="yes"/>
 <layer number="26" name="bNames" color="7" fill="1" visible="yes" active="yes"/>
-<layer number="27" name="tValues" color="7" fill="1" visible="no" active="yes"/>
+<layer number="27" name="tValues" color="7" fill="1" visible="yes" active="yes"/>
 <layer number="28" name="bValues" color="7" fill="1" visible="yes" active="yes"/>
 <layer number="29" name="tStop" color="7" fill="3" visible="no" active="yes"/>
@@
 <wire x1="25.4" y1="74.13625" x2="25.4" y2="76.67625" width="0.4064" layer="114"/>
 <wire x1="15.5575" y1="97.94875" x2="13.0175" y2="97.94875" width="0.4064" layer="114"/>
+<dimension x1="-1.27" y1="113.9825" x2="8.5725" y2="103.1875" x3="-7.62" y3="108.585" layer="21" dtype="vertical"/>
 </plain>
 <attributes>
@@
 </autorouter>
 <elements>
-<element name="DD2" library="Speccy" package="PGA-84-B" value="EPM7128-J84" x="64.77" y="31.90875" smashed="yes">
+<element name="DD2" library="Speccy" package="PGA-84-B" value="EPM7128SLC84-15" x="64.77" y="31.90875" smashed="yes">
 <attribute name="NAME" x="60.96" y="11.27125" size="1.778" layer="25"/>
 <attribute name="VALUE" x="66.9925" y="11.27125" size="1.778" layer="27"/>
@@
 </element>
 <element name="R2Y" library="rcl" package="R0805" value="2k" x="72.0725" y="84.29625" smashed="yes" rot="MR270">
-<attribute name="NAME" x="76.5175" y="93.18625" size="1.27" layer="26" rot="MR270"/>
+<attribute name="NAME" x="75.2475" y="93.50375" size="1.27" layer="26" rot="MR270"/>
 <attribute name="VALUE" x="72.7075" y="96.04375" size="1.27" layer="28" rot="MR270"/>
 </element>
@@
 <attribute name="VALUE" x="152.781" y="3.58775" size="1.778" layer="27" rot="R180"/>
 </element>
-<element name="DD11" library="Speccy" package="DIL14" value="74LS04N" x="17.4625" y="54.45125"/>
+<element name="DD11" library="Speccy" package="DIL14" value="К555ЛН1" x="17.4625" y="54.45125"/>
 <element name="-R3" library="rcl" package="R0805" value="360" x="13.6525" y="55.40375" smashed="yes" rot="MR180">
 <attribute name="NAME" x="13.6525" y="54.13375" size="1.27" layer="26" rot="MR180"/>
@@
 <attribute name="VALUE" x="20.0025" y="52.86375" size="1.27" layer="28" rot="MR0"/>
 </element>
-<element name="DA1" library="cxa1645" package="DIL24-4" value="CXA1645" x="14.9225" y="76.04125" smashed="yes" rot="R270">
+<element name="DA1" library="cxa1645" package="DIL24-4" value="CXA1645P" x="14.9225" y="76.04125" smashed="yes" rot="R270">
 <attribute name="NAME" x="12.7" y="93.91015" size="1.778" layer="25" ratio="10"/>
 <attribute name="VALUE" x="10.00125" y="91.8718" size="1.778" layer="27" ratio="10"/>
@@
 <attribute name="VALUE" x="17.4625" y="62.07125" size="1.27" layer="28" rot="MR0"/>
 </element>
-<element name="R6P" library="rcl" package="R1206" value="47k" x="24.4475" y="62.07125" smashed="yes" rot="MR0">
+<element name="R6P" library="rcl" package="R0805" value="47k" x="24.4475" y="62.07125" smashed="yes" rot="MR0">
 <attribute name="NAME" x="26.67" y="59.84875" size="1.27" layer="26" rot="MR180"/>
 <attribute name="VALUE" x="26.9875" y="57.62625" size="1.27" layer="28" rot="MR180"/>
@@
 <attribute name="VALUE" x="112.7125" y="77.94625" size="1.27" layer="28" rot="MR270"/>
 </element>
-<element name="R2" library="rcl" package="R1206" value="" x="157.7975" y="99.53625" smashed="yes" rot="MR180">
+<element name="R2" library="rcl" package="R1206" value="0" x="157.7975" y="99.53625" smashed="yes" rot="MR180">
 <attribute name="NAME" x="154.6225" y="97.63125" size="1.27" layer="26" rot="MR180"/>
 <attribute name="VALUE" x="156.5275" y="102.07625" size="1.27" layer="28" rot="MR180"/>
 </element>
-<element name="DD12" library="Speccy" package="DIL14O" value="74LS74O" x="58.1025" y="66.19875" smashed="yes" rot="R180">
+<element name="DD12" library="Speccy" package="DIL14O" value="К155ТМ2" x="58.1025" y="66.19875" smashed="yes" rot="R180">
 <attribute name="NAME" x="58.70575" y="59.436" size="1.27" layer="25" ratio="10"/>
 <attribute name="VALUE" x="64.516" y="58.89625" size="1.27" layer="27" ratio="10" rot="R180"/>
@@
 <wire x1="13.335" y1="73.81875" x2="12.3825" y2="74.77125" width="0.4064" layer="1"/>
 <wire x1="12.3825" y1="74.77125" x2="9.8425" y2="74.77125" width="0.4064" layer="1"/>
-<wire x1="25.8695" y1="62.07125" x2="25.7175" y2="64.45925" width="0.4064" layer="16"/>
+<wire x1="25.3975" y1="62.07125" x2="25.7175" y2="64.45925" width="0.4064" layer="16"/>
 <wire x1="25.7175" y1="64.45925" x2="25.7175" y2="65.56375" width="0.4064" layer="16"/>
 <wire x1="22.2885" y1="35.21075" x2="22.2885" y2="39.116" width="0.4064" layer="1"/>
@@
 <via x="4.445" y="13.335" extent="1-16" drill="0.8" diameter="2.1844"/>
 <wire x1="4.445" y1="13.335" x2="3.81" y2="13.97" width="0.8128" layer="1"/>
-<wire x1="3.81" y1="13.97" x2="3.81" y2="96.2025" width="0.8128" layer="1"/>
+<wire x1="3.81" y1="13.97" x2="3.81" y2="94.615" width="0.8128" layer="1"/>
+<wire x1="3.81" y1="94.615" x2="3.81" y2="96.2025" width="0.8128" layer="1"/>
 <wire x1="3.81" y1="96.2025" x2="5.715" y2="98.1075" width="0.8128" layer="1"/>
 <via x="5.715" y="98.1075" extent="1-16" drill="0.8" diameter="2.1844"/>
@@
 <contactref element="CX1" pad="2"/>
 <wire x1="77.26" y1="105.29125" x2="75.25" y2="103.70375" width="0.8128" layer="16"/>
-<wire x1="77.1525" y1="88.10625" x2="77.1525" y2="90.64625" width="0.8128" layer="16"/>
+<wire x1="77.1525" y1="88.10625" x2="77.1525" y2="89.05875" width="0.8128" layer="16"/>
 <wire x1="62.23" y1="19.20875" x2="62.23" y2="20.32" width="1.016" layer="16"/>
 <wire x1="62.23" y1="20.32" x2="61.43625" y2="20.6375" width="0.4064" layer="16"/>
@@
 <wire x1="12.22375" y1="25.87625" x2="14.176375" y2="25.87625" width="0.3048" layer="1"/>
 <contactref element="C1" pad="-"/>
-<wire x1="77.1525" y1="90.64625" x2="75.91425" y2="91.8845" width="0.8128" layer="16"/>
-<wire x1="75.91425" y1="91.8845" x2="72.39" y2="91.8845" width="0.8128" layer="16"/>
+<wire x1="77.1525" y1="89.05875" x2="75.27925" y2="91.8845" width="0.8128" layer="16"/>
+<wire x1="75.27925" y1="91.8845" x2="72.39" y2="91.8845" width="0.8128" layer="16"/>
 <wire x1="72.39" y1="91.8845" x2="70.1675" y2="91.8845" width="0.8128" layer="16"/>
 <wire x1="75.25" y1="103.70375" x2="67.6275" y2="96.08125" width="0.8128" layer="16"/>
@@
 <wire x1="69.4055" y1="91.8845" x2="70.1675" y2="91.8845" width="0.8128" layer="16"/>
 <wire x1="72.39" y1="93.03" x2="72.39" y2="91.8845" width="0.8128" layer="16"/>
-<wire x1="7.46125" y1="42.545" x2="9.2075" y2="38.25625" width="0" layer="19" extent="1-1"/>
+<wire x1="5.715" y1="94.615" x2="3.81" y2="94.615" width="0.8128" layer="1"/>
+<wire x1="77.1525" y1="105.0925" x2="80.01" y2="107.95" width="0.8128" layer="1"/>
+<via x="76.5175" y="91.1225" extent="1-16" drill="0.8" diameter="2.1844"/>
+<wire x1="77.1525" y1="88.265" x2="76.5175" y2="91.1225" width="0.8128" layer="1"/>
+<via x="26.035" y="67.945" extent="1-16" drill="0.8" diameter="2.1844"/>
+<wire x1="25.7175" y1="65.7225" x2="26.035" y2="67.945" width="0.8128" layer="1"/>
+<wire x1="26.035" y1="67.945" x2="25.7175" y2="65.7225" width="0.8128" layer="16"/>
+<wire x1="80.01" y1="107.79125" x2="80.01" y2="107.95" width="0" layer="19" extent="1-16"/>
+<wire x1="77.1525" y1="88.265" x2="77.1525" y2="88.10625" width="0" layer="19" extent="1-1"/>
+<wire x1="25.7175" y1="65.7225" x2="25.7175" y2="65.56375" width="0" layer="19" extent="1-16"/>
+<wire x1="9.2075" y1="38.25625" x2="7.46125" y2="42.545" width="0" layer="19" extent="1-1"/>
 </signal>
 <signal name="D1">
@@
 <contactref element="DD11" pad="13"/>
 <wire x1="12.3825" y1="58.26125" x2="12.7025" y2="55.40375" width="1.016" layer="16"/>
-<wire x1="24.4475" y1="53.18125" x2="13.6525" y2="53.18125" width="0.4064" layer="16"/>
-<wire x1="13.6525" y1="53.18125" x2="12.7" y2="54.13375" width="0.4064" layer="16"/>
+<wire x1="24.765" y1="53.49875" x2="13.335" y2="53.49875" width="0.4064" layer="16"/>
+<wire x1="13.335" y1="53.49875" x2="12.7" y2="54.13375" width="0.4064" layer="16"/>
 <wire x1="12.7" y1="54.13375" x2="12.7" y2="55.08375" width="0.4064" layer="16"/>
 <wire x1="12.7" y1="55.08375" x2="12.7025" y2="55.40375" width="0.4064" layer="16"/>
 <contactref element="Z2" pad="1"/>
-<wire x1="24.4475" y1="53.18125" x2="30.7975" y2="59.53125" width="0.4064" layer="16"/>
+<wire x1="24.765" y1="53.49875" x2="30.7975" y2="59.53125" width="0.4064" layer="16"/>
 <wire x1="30.7975" y1="59.53125" x2="30.7975" y2="65.43675" width="0.4064" layer="16"/>
 <wire x1="30.7975" y1="65.43675" x2="28.575" y2="65.75425" width="0.4064" layer="16"/>
@@
 <contactref element="C5P" pad="2"/>
 <contactref element="R6P" pad="2"/>
-<wire x1="20.0025" y1="62.07125" x2="23.0255" y2="62.07125" width="0.4064" layer="16"/>
+<wire x1="20.0025" y1="62.07125" x2="23.4975" y2="62.07125" width="0.4064" layer="16"/>
 <wire x1="20.0025" y1="62.07125" x2="17.30375" y2="62.07125" width="0.6096" layer="16"/>
 <wire x1="17.30375" y1="62.07125" x2="16.3225" y2="63.0525" width="0.6096" layer="16"/>
@@
 <via x="76.835" y="96.36125" extent="1-16" drill="3.2" diameter="5"/>
 </signal>
+<signal name="N$61">
+<via x="6.985" y="107.47375" extent="1-16" drill="3.2" diameter="5"/>
+</signal>
 <signal name="N$26">
 <via x="165.4175" y="88.10625" extent="1-16" drill="3.2" diameter="5"/>
-<via x="6.985" y="107.47375" extent="1-16" drill="3.2" diameter="5"/>
 </signal>
 <signal name="V_OUT">

Commit message: .....
Parts:
- -R3, R112, R27, R34: value 360 -> 390
- C8P, C8P1, C8P2, C9, C9P, CP2: device Speccy:E2,5-5 -> Speccy:E2,5-6
- DA2: value AP1117 -> L1117-3.3
- moved C9 0.71 mm to (28.3, 42.7)
- moved R_B 0.64 mm to (43.5, 8.41)
- moved R26 0.63 mm to (10.6, 23.8)
- moved R_G 0.63 mm to (48.6, 8.41)
- moved R16 0.32 mm to (32.7, 43.0)
- moved R_R 0.32 mm to (53.3, 8.41)
- moved R_SY 0.32 mm to (58.4, 8.41)
Routing:
- net GND: track 1243.6 -> 1246.6 mm
- net N$16: track 42.8 -> 43.6 mm
- net N$14: track 28.0 -> 28.7 mm
- net N$13: track 44.9 -> 45.6 mm
Other:
- board text added: "SD Card"

Commit message: .....
Parts:
- R25: value 1k -> 150
Changed lines of the file:
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@@
 DIP 128KB Y</text>
 <text x="21.2725" y="6.0325" size="1.9304" layer="1" font="vector" ratio="15">SD Card</text>
+<rectangle x1="23.1775" y1="19.685" x2="27.6225" y2="24.4475" layer="16"/>
 </plain>
 <attributes>
@@
 <attribute name="VALUE" x="8.00875" y="32.1625" size="1.27" layer="27" rot="R180"/>
 </element>
-<element name="R25" library="rcl" package="R0805" value="1k" x="9.2075" y="37.30625" smashed="yes" rot="R270">
+<element name="R25" library="rcl" package="R0805" value="150" x="9.2075" y="37.30625" smashed="yes" rot="R270">
 <attribute name="NAME" x="7.46125" y="39.0525" size="1.27" layer="25" rot="R180"/>
 <attribute name="VALUE" x="7.46125" y="37.1475" size="1.27" layer="27" rot="R180"/>

Commit message: .....
Parts:
- DD7: value MEGA16-P -> ATMEGA32-P
Changed lines of the file:
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@@
 </element>
 <element name="DD6" library="Speccy" package="DIL28+6" value="62256" x="95.885" y="24.28875" smashed="yes" rot="R90">
-<attribute name="NAME" x="89.2175" y="4.60375" size="1.778" layer="25" ratio="10"/>
-<attribute name="VALUE" x="95.5675" y="4.61645" size="1.778" layer="27" ratio="10"/>
+<attribute name="NAME" x="89.2175" y="4.28625" size="1.778" layer="25" ratio="10"/>
+<attribute name="VALUE" x="95.5675" y="4.29895" size="1.778" layer="27" ratio="10"/>
 </element>
-<element name="DD7" library="atmel" package="DIL40" value="MEGA16-P" x="94.2975" y="85.56625" smashed="yes" rot="R90">
+<element name="DD7" library="atmel" package="DIL40" value="ATMEGA32-P" x="94.2975" y="85.56625" smashed="yes" rot="R90">
 <attribute name="OC_NEWARK" value="01M6885" x="137.4775" y="124.93625" size="1.778" layer="27" rot="R90" display="off"/>
 <attribute name="MPN" value="ATMEGA16-16PU" x="137.4775" y="124.93625" size="1.778" layer="27" rot="R90" display="off"/>
 <attribute name="MF" value="" x="137.4775" y="124.93625" size="1.778" layer="27" rot="R90" display="off"/>
 <attribute name="OC_FARNELL" value="9171142" x="137.4775" y="124.93625" size="1.778" layer="27" rot="R90" display="off"/>
-<attribute name="NAME" x="92.3925" y="57.94375" size="1.778" layer="25" ratio="10" rot="R180"/>
-<attribute name="VALUE" x="100.0125" y="55.41645" size="1.778" layer="27" ratio="10" rot="R180"/>
+<attribute name="NAME" x="96.8375" y="58.26125" size="1.778" layer="25" ratio="10" rot="R180"/>
+<attribute name="VALUE" x="102.235" y="56.05145" size="1.778" layer="27" ratio="10" rot="R180"/>
 </element>
 <element name="DD1" library="zilog" package="DIL40" value="Z80" x="120.65" y="85.56625" smashed="yes" rot="R270">

Commit message: .....
Parts:
- added C20P: 47, rcl:C0805
- DD10, DD4, DD5: value 74HC245N -> 74HCT245N
- R5P: value 16k* -> 16k 1%
- R_B, R_G, R_R, R_SY: value (none) -> 1k
Connections:
- new net N$62: C20P.2, DA1.6
- net FC: now also C20P.1; no longer DA1.6
Routing:
- net N$62: track 0.00 -> 3.37 mm
- net FC: track 53.2 -> 55.9 mm
- net SPEAKER: track 215.0 -> 215.9 mm
Other:
- board text added: "r1.01"
Changed lines of the file:
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@@
 <text x="21.2725" y="6.0325" size="1.9304" layer="1" font="vector" ratio="15">SD Card</text>
 <rectangle x1="23.1775" y1="19.685" x2="27.6225" y2="24.4475" layer="16"/>
+<text x="71.4375" y="8.89" size="1.9304" layer="1" font="vector" ratio="15">r1.01</text>
 </plain>
 <attributes>
@@
 <attribute name="VALUE" x="17.145" y="48.26" size="1.27" layer="28" rot="MR270"/>
 </element>
-<element name="DD4" library="Speccy" package="DIL20" value="74HC245N" x="111.77" y="16.67875" smashed="yes" rot="R90">
+<element name="DD4" library="Speccy" package="DIL20" value="74HCT245N" x="111.77" y="16.67875" smashed="yes" rot="R90">
 <attribute name="NAME" x="113.548" y="3.59775" size="1.27" layer="25" rot="R180"/>
 <attribute name="VALUE" x="107.54725" y="29.7715" size="1.27" layer="27"/>
 </element>
-<element name="DD5" library="Speccy" package="DIL20" value="74HC245N" x="126.245" y="16.68125" smashed="yes" rot="R90">
+<element name="DD5" library="Speccy" package="DIL20" value="74HCT245N" x="126.245" y="16.68125" smashed="yes" rot="R90">
 <attribute name="NAME" x="128.023" y="3.60025" size="1.27" layer="25" rot="R180"/>
 <attribute name="VALUE" x="122.47225" y="29.9015" size="1.27" layer="27"/>
 </element>
-<element name="DD10" library="Speccy" package="DIL20" value="74HC245N" x="145.0875" y="54.28875" smashed="yes" rot="R180">
+<element name="DD10" library="Speccy" package="DIL20" value="74HCT245N" x="145.0875" y="54.28875" smashed="yes" rot="R180">
 <attribute name="NAME" x="158.24575" y="53.711" size="1.27" layer="25"/>
 <attribute name="VALUE" x="158.1885" y="51.69275" size="1.27" layer="27"/>
@@
 <attribute name="VALUE" x="15.5575" y="67.15125" size="1.27" layer="28" rot="MR0"/>
 </element>
-<element name="R_R" library="Speccy" package="RTRIM3296W" value="" x="53.34" y="8.41375" smashed="yes" rot="R180">
+<element name="R_R" library="Speccy" package="RTRIM3296W" value="1k" x="53.34" y="8.41375" smashed="yes" rot="R180">
 <attribute name="NAME" x="51.38" y="2.49125" size="1.27" layer="25"/>
 <attribute name="VALUE" x="49.39" y="12.91375" size="1.27" layer="27" rot="R270"/>
 </element>
-<element name="R_G" library="Speccy" package="RTRIM3296W" value="" x="48.5775" y="8.41375" smashed="yes" rot="R180">
+<element name="R_G" library="Speccy" package="RTRIM3296W" value="1k" x="48.5775" y="8.41375" smashed="yes" rot="R180">
 <attribute name="NAME" x="46.935" y="2.49125" size="1.27" layer="25"/>
 <attribute name="VALUE" x="44.6275" y="12.91375" size="1.27" layer="27" rot="R270"/>
 </element>
-<element name="R_B" library="Speccy" package="RTRIM3296W" value="" x="43.4975" y="8.41375" smashed="yes" rot="R180">
+<element name="R_B" library="Speccy" package="RTRIM3296W" value="1k" x="43.4975" y="8.41375" smashed="yes" rot="R180">
 <attribute name="NAME" x="41.855" y="2.49125" size="1.27" layer="25"/>
 <attribute name="VALUE" x="39.5475" y="12.91375" size="1.27" layer="27" rot="R270"/>
@@
 <attribute name="VALUE" x="7.77875" y="22.225" size="1.27" layer="28" rot="MR90"/>
 </element>
-<element name="R_SY" library="Speccy" package="RTRIM3296W" value="" x="58.42" y="8.41375" smashed="yes" rot="R180">
+<element name="R_SY" library="Speccy" package="RTRIM3296W" value="1k" x="58.42" y="8.41375" smashed="yes" rot="R180">
 <attribute name="NAME" x="56.1425" y="2.49125" size="1.27" layer="25"/>
 <attribute name="VALUE" x="54.47" y="12.91375" size="1.27" layer="27" rot="R270"/>
@@
 <attribute name="VALUE" x="68.7705" y="98.39325" size="1.27" layer="27" ratio="10"/>
 </element>
-<element name="R5P" library="rcl" package="M1206" value="16k*" x="15.5575" y="74.77125" smashed="yes" rot="MR180">
+<element name="R5P" library="rcl" package="M1206" value="16k 1%" x="15.5575" y="74.77125" smashed="yes" rot="MR180">
 <attribute name="NAME" x="17.78" y="76.35875" size="1.27" layer="26" rot="MR0"/>
 <attribute name="VALUE" x="17.78" y="71.91375" size="1.27" layer="28" rot="MR0"/>
@@
 </element>
 <element name="C1" library="Speccy" package="E3,5-8" value="" x="70.1675" y="93.6625" rot="R270"/>
+<element name="C20P" library="rcl" package="C0805" value="47" x="6.6675" y="76.67625" smashed="yes" rot="R90">
+<attribute name="NAME" x="5.715" y="79.21625" size="1.27" layer="25" rot="R90"/>
+<attribute name="VALUE" x="7.62" y="79.53375" size="1.27" layer="27" rot="R90"/>
+</element>
 </elements>
 <signals>
@@
 <wire x1="54.9275" y1="4.60375" x2="54.2925" y2="3.96875" width="0.4064" layer="1"/>
 <wire x1="54.2925" y1="3.96875" x2="40.64" y2="3.96875" width="0.4064" layer="1"/>
-<wire x1="6.0325" y1="34.13125" x2="6.0325" y2="90.64625" width="0.4064" layer="1"/>
-<wire x1="6.0325" y1="90.64625" x2="7.9375" y2="92.55125" width="0.4064" layer="1"/>
+<wire x1="5.715" y1="90.32875" x2="7.9375" y2="92.55125" width="0.4064" layer="1"/>
 <wire x1="7.9375" y1="92.55125" x2="21.9075" y2="92.55125" width="0.4064" layer="1"/>
 <wire x1="21.9075" y1="92.55125" x2="25.4" y2="89.05875" width="0.4064" layer="1"/>
@@
 <wire x1="7.3025" y1="25.24125" x2="10.16" y2="28.09875" width="0.4064" layer="1"/>
 <wire x1="10.16" y1="28.09875" x2="10.16" y2="30.00375" width="0.4064" layer="1"/>
-<wire x1="10.16" y1="30.00375" x2="6.0325" y2="34.13125" width="0.4064" layer="1"/>
+<wire x1="10.16" y1="30.00375" x2="5.78939375" y2="34.37435625" width="0.4064" layer="1"/>
+<wire x1="5.78939375" y1="34.37435625" x2="5.715" y2="34.44875" width="0.4064" layer="1"/>
 <wire x1="54.9275" y1="4.60375" x2="54.9275" y2="13.335" width="0.4064" layer="1"/>
 <wire x1="54.9275" y1="13.335" x2="53.6575" y2="14.605" width="0.4064" layer="1"/>
@@
 <wire x1="10.4775" y1="14.9225" x2="8.5725" y2="14.9225" width="0.4064" layer="1"/>
 <wire x1="8.5725" y1="14.9225" x2="7.3025" y2="16.1925" width="0.4064" layer="1"/>
+<wire x1="5.715" y1="90.32875" x2="5.715" y2="79.797709375" width="0.4064" layer="1"/>
+<wire x1="5.715" y1="79.797709375" x2="5.64060625" y2="79.61810625" width="0.4064" layer="1" curve="-44.999502"/>
+<wire x1="5.64060625" y1="79.61810625" x2="5.08" y2="79.0575" width="0.4064" layer="1"/>
+<wire x1="5.08" y1="73.66" x2="5.715" y2="73.025" width="0.4064" layer="1"/>
+<wire x1="5.715" y1="73.025" x2="5.715" y2="34.553959375" width="0.4064" layer="1"/>
+<wire x1="5.715" y1="34.553959375" x2="5.78939375" y2="34.37435625" width="0.4064" layer="1" curve="44.999502"/>
+<wire x1="5.08" y1="79.0575" x2="5.08" y2="73.66" width="0.4064" layer="1"/>
 </signal>
 <signal name="G">
@@
 </signal>
 <signal name="FC">
-<contactref element="DA1" pad="6"/>
 <contactref element="DD12" pad="9"/>
 <via x="45.085" y="68.73875" extent="1-16" drill="0.8" diameter="2.1844"/>
@@
 <wire x1="53.0225" y1="64.61125" x2="48.895" y2="68.73875" width="0.4064" layer="16"/>
 <wire x1="48.895" y1="68.73875" x2="45.085" y2="68.73875" width="0.4064" layer="16"/>
-<wire x1="9.8425" y1="77.31125" x2="16.8275" y2="77.31125" width="0.4064" layer="1"/>
-<wire x1="16.8275" y1="77.31125" x2="18.0975" y2="76.04125" width="0.4064" layer="1"/>
 <wire x1="18.0975" y1="76.04125" x2="21.59" y2="76.04125" width="0.3048" layer="1"/>
 <wire x1="21.59" y1="76.04125" x2="22.5425" y2="75.08875" width="0.4064" layer="1"/>
 <wire x1="22.5425" y1="75.08875" x2="22.5425" y2="70.8025" width="0.4064" layer="1"/>
 <wire x1="22.5425" y1="70.8025" x2="23.65375" y2="69.69125" width="0.4064" layer="1"/>
+<contactref element="C20P" pad="1"/>
+<wire x1="18.0975" y1="76.04125" x2="11.58875" y2="76.04125" width="0.4064" layer="1"/>
+<wire x1="11.58875" y1="76.04125" x2="7.9375" y2="76.04125" width="0.3048" layer="1"/>
+<wire x1="7.9375" y1="76.04125" x2="6.6675" y2="75.72625" width="0.3048" layer="1"/>
 </signal>
 <signal name="N$35">
@@
 <wire x1="170.4975" y1="1.5875" x2="170.4975" y2="3.175" width="0.6096" layer="1"/>
 </signal>
+<signal name="N$62">
+<contactref element="C20P" pad="2"/>
+<contactref element="DA1" pad="6"/>
+<wire x1="9.8425" y1="77.31125" x2="6.82375" y2="77.31125" width="0.3048" layer="1"/>
+<wire x1="6.82375" y1="77.31125" x2="6.6675" y2="77.62625" width="0.3048" layer="1"/>
+</signal>
 </signals>
