File: Speccy2007_128K_Ljubitel.brd (EAGLE design)
At the start: 168.6 x 112.4 mm, 119 parts, among them X1 5V, X2 SCART-F, X3 PS/2 KB, X4 SD Card, X5 ByteBlaster, X6 AVRISP

Commit message: .....
Parts:
- J1: value (none) -> 0
- X3P: value (none) -> KB
Other:
- board text added: "C"
- board text added: "D"
- board text added: "G"
- board text added: "V"
Changed lines of the file:
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@@
 <rectangle x1="23.1775" y1="19.685" x2="27.6225" y2="24.4475" layer="16"/>
 <text x="71.4375" y="8.89" size="1.9304" layer="1" font="vector" ratio="15">r1.01</text>
+<text x="166.0525" y="91.44" size="1.27" layer="21" font="vector" ratio="15">G</text>
+<text x="163.5125" y="91.44" size="1.27" layer="21" font="vector" ratio="15">V</text>
+<text x="160.9725" y="91.44" size="1.27" layer="21" font="vector" ratio="15">D</text>
+<text x="158.4325" y="91.44" size="1.27" layer="21" font="vector" ratio="15">C</text>
 </plain>
 <attributes>
@@
 </element>
 <element name="X3" library="Speccy" package="MINI-DIN6" value="PS/2 KB" x="162.56" y="113.18875" smashed="yes">
-<attribute name="NAME" x="160.3375" y="98.90125" size="1.27" layer="25"/>
-<attribute name="VALUE" x="158.115" y="96.99625" size="1.27" layer="27"/>
+<attribute name="NAME" x="156.5275" y="98.90125" size="1.27" layer="25"/>
+<attribute name="VALUE" x="160.02" y="98.90125" size="1.27" layer="27"/>
 </element>
 <element name="DD3" library="Speccy" package="DIL32" value="621024" x="145.7325" y="24.28875" smashed="yes" rot="R90">
@@
 <attribute name="VALUE" x="28.09875" y="81.12125" size="1.27" layer="28" rot="MR180"/>
 </element>
-<element name="J1" library="rcl" package="M1206" value="" x="110.1725" y="76.67625" smashed="yes" rot="MR270">
+<element name="J1" library="rcl" package="M1206" value="0" x="110.1725" y="76.67625" smashed="yes" rot="MR270">
 <attribute name="NAME" x="108.2675" y="76.04125" size="1.27" layer="26" rot="MR0"/>
 <attribute name="VALUE" x="112.7125" y="77.94625" size="1.27" layer="28" rot="MR270"/>
@@
 <attribute name="VALUE" x="15.875" y="80.01" size="1.27" layer="28" rot="MR0"/>
 </element>
-<element name="X3P" library="con-lstb" package="MA04-1" value="" x="162.56" y="94.615" smashed="yes">
+<element name="X3P" library="con-lstb" package="MA04-1" value="KB" x="162.56" y="94.615" smashed="yes">
 <attribute name="OC_NEWARK" value="unknown" x="162.56" y="94.615" size="1.778" layer="27" display="off"/>
 <attribute name="MPN" value="" x="162.56" y="94.615" size="1.778" layer="27" display="off"/>
 <attribute name="MF" value="" x="162.56" y="94.615" size="1.778" layer="27" display="off"/>
 <attribute name="OC_FARNELL" value="unknown" x="162.56" y="94.615" size="1.778" layer="27" display="off"/>
-<attribute name="NAME" x="164.1475" y="98.4885" size="1.27" layer="25" ratio="10"/>
-<attribute name="VALUE" x="163.195" y="96.266" size="1.27" layer="27" ratio="10"/>
+<attribute name="NAME" x="156.21" y="89.281" size="1.27" layer="25" ratio="10"/>
+<attribute name="VALUE" x="160.655" y="89.281" size="1.27" layer="27" ratio="10"/>
 </element>
 <element name="CE2" library="rcl" package="C0805" value="100n" x="74.6125" y="41.5925" smashed="yes" rot="MR270">

Commit message: fix pal 1
Parts:
- added J2: 0, rcl:R0805
- C1: value (none) -> 1000mfx6.3v
- VT1: value BC337(KT503) -> KT503Г(BC337)
- Z2: value 4.43Mhz -> 8867.232KHz/4..20pf
- moved Z2 1.77 mm to (35.2, 64.1)
- moved C4P 0.95 mm to (13.7, 68.7)
- moved R5P 0.64 mm to (15.6, 75.4)
- moved C6P 0.45 mm to (24.1, 65.9)
- moved R6P 0.32 mm to (24.1, 62.1)
- renumbered R3 to RF1
Connections:
- net FC: now also J2.2
- net FCI: now also J2.1
Routing:
- net +5V: track 860.7 -> 884.0 mm, vias 3 -> 4
- net FCI: track 44.9 -> 48.1 mm
- net N$45: track 33.2 -> 34.6 mm
- net N$44: track 17.0 -> 18.2 mm
- net CLK: track 151.3 -> 152.3 mm
- net GND: track 1246.6 -> 1247.5 mm
