File: Speccy2007_128K_Ljubitel.sch (EAGLE design)
At the start: 100 parts, among them X2 SCART-F, X5 ByteBlaster, X6 AVRISP

Commit message: .
Parts:
- R_B, R_G, R_R, R_SY: device resistor:R-TRIMM3296W -> Speccy:R-TRIMM3296W
Changed lines of the file:
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@@
 <grid distance="100" unitdist="mil" unit="mil" style="lines" multiple="1" display="yes" altdistance="0.01" altunitdist="inch" altunit="inch"/>
 <layers>
-<layer number="1" name="Top" color="4" fill="1" visible="yes" active="no"/>
-<layer number="2" name="Route2" color="1" fill="3" visible="yes" active="no"/>
-<layer number="3" name="Route3" color="4" fill="3" visible="yes" active="no"/>
-<layer number="4" name="Route4" color="1" fill="4" visible="yes" active="no"/>
-<layer number="5" name="Route5" color="4" fill="4" visible="yes" active="no"/>
-<layer number="6" name="Route6" color="1" fill="8" visible="yes" active="no"/>
-<layer number="7" name="Route7" color="4" fill="8" visible="yes" active="no"/>
-<layer number="8" name="Route8" color="1" fill="2" visible="yes" active="no"/>
-<layer number="9" name="Route9" color="4" fill="2" visible="yes" active="no"/>
-<layer number="10" name="Route10" color="1" fill="7" visible="yes" active="no"/>
-<layer number="11" name="Route11" color="4" fill="7" visible="yes" active="no"/>
-<layer number="12" name="Route12" color="1" fill="5" visible="yes" active="no"/>
-<layer number="13" name="Route13" color="4" fill="5" visible="yes" active="no"/>
-<layer number="14" name="Route14" color="1" fill="6" visible="yes" active="no"/>
-<layer number="15" name="Route15" color="4" fill="6" visible="yes" active="no"/>
-<layer number="16" name="Bottom" color="1" fill="1" visible="yes" active="no"/>
-<layer number="17" name="Pads" color="2" fill="1" visible="yes" active="no"/>
-<layer number="18" name="Vias" color="2" fill="1" visible="yes" active="no"/>
-<layer number="19" name="Unrouted" color="6" fill="1" visible="yes" active="no"/>
-<layer number="20" name="Dimension" color="15" fill="1" visible="yes" active="no"/>
-<layer number="21" name="tPlace" color="7" fill="1" visible="yes" active="no"/>
-<layer number="22" name="bPlace" color="7" fill="1" visible="yes" active="no"/>
-<layer number="23" name="tOrigins" color="15" fill="1" visible="yes" active="no"/>
-<layer number="24" name="bOrigins" color="15" fill="1" visible="yes" active="no"/>
-<layer number="25" name="tNames" color="7" fill="1" visible="yes" active="no"/>
-<layer number="26" name="bNames" color="7" fill="1" visible="yes" active="no"/>
-<layer number="27" name="tValues" color="7" fill="1" visible="yes" active="no"/>
-<layer number="28" name="bValues" color="7" fill="1" visible="yes" active="no"/>
+<layer number="1" name="Top" color="4" fill="1" visible="no" active="no"/>
+<layer number="2" name="Route2" color="1" fill="3" visible="no" active="no"/>
+<layer number="3" name="Route3" color="4" fill="3" visible="no" active="no"/>
+<layer number="4" name="Route4" color="1" fill="4" visible="no" active="no"/>
+<layer number="5" name="Route5" color="4" fill="4" visible="no" active="no"/>
+<layer number="6" name="Route6" color="1" fill="8" visible="no" active="no"/>
+<layer number="7" name="Route7" color="4" fill="8" visible="no" active="no"/>
+<layer number="8" name="Route8" color="1" fill="2" visible="no" active="no"/>
+<layer number="9" name="Route9" color="4" fill="2" visible="no" active="no"/>
+<layer number="10" name="Route10" color="1" fill="7" visible="no" active="no"/>
+<layer number="11" name="Route11" color="4" fill="7" visible="no" active="no"/>
+<layer number="12" name="Route12" color="1" fill="5" visible="no" active="no"/>
+<layer number="13" name="Route13" color="4" fill="5" visible="no" active="no"/>
+<layer number="14" name="Route14" color="1" fill="6" visible="no" active="no"/>
+<layer number="15" name="Route15" color="4" fill="6" visible="no" active="no"/>
+<layer number="16" name="Bottom" color="1" fill="1" visible="no" active="no"/>
+<layer number="17" name="Pads" color="2" fill="1" visible="no" active="no"/>
+<layer number="18" name="Vias" color="2" fill="1" visible="no" active="no"/>
+<layer number="19" name="Unrouted" color="6" fill="1" visible="no" active="no"/>
+<layer number="20" name="Dimension" color="15" fill="1" visible="no" active="no"/>
+<layer number="21" name="tPlace" color="7" fill="1" visible="no" active="no"/>
+<layer number="22" name="bPlace" color="7" fill="1" visible="no" active="no"/>
+<layer number="23" name="tOrigins" color="15" fill="1" visible="no" active="no"/>
+<layer number="24" name="bOrigins" color="15" fill="1" visible="no" active="no"/>
+<layer number="25" name="tNames" color="7" fill="1" visible="no" active="no"/>
+<layer number="26" name="bNames" color="7" fill="1" visible="no" active="no"/>
+<layer number="27" name="tValues" color="7" fill="1" visible="no" active="no"/>
+<layer number="28" name="bValues" color="7" fill="1" visible="no" active="no"/>
 <layer number="29" name="tStop" color="7" fill="3" visible="no" active="no"/>
 <layer number="30" name="bStop" color="7" fill="6" visible="no" active="no"/>
@@
 <layer number="35" name="tGlue" color="7" fill="4" visible="no" active="no"/>
 <layer number="36" name="bGlue" color="7" fill="5" visible="no" active="no"/>
-<layer number="37" name="tTest" color="7" fill="1" visible="yes" active="no"/>
-<layer number="38" name="bTest" color="7" fill="1" visible="yes" active="no"/>
+<layer number="37" name="tTest" color="7" fill="1" visible="no" active="no"/>
+<layer number="38" name="bTest" color="7" fill="1" visible="no" active="no"/>
 <layer number="39" name="tKeepout" color="4" fill="11" visible="no" active="no"/>
 <layer number="40" name="bKeepout" color="1" fill="11" visible="no" active="no"/>
@@
 <layer number="44" name="Drills" color="7" fill="1" visible="no" active="no"/>
 <layer number="45" name="Holes" color="7" fill="1" visible="no" active="no"/>
-<layer number="46" name="Milling" color="3" fill="1" visible="yes" active="no"/>
-<layer number="47" name="Measures" color="7" fill="1" visible="yes" active="no"/>
-<layer number="48" name="Document" color="7" fill="1" visible="yes" active="no"/>
-<layer number="49" name="Reference" color="7" fill="1" visible="yes" active="no"/>
-<layer number="50" name="dxf" color="7" fill="1" visible="yes" active="no"/>
-<layer number="51" name="tDocu" color="7" fill="1" visible="yes" active="no"/>
-<layer number="52" name="bDocu" color="7" fill="1" visible="yes" active="no"/>
-<layer number="53" name="tGND_GNDA" color="7" fill="9" visible="yes" active="no"/>
-<layer number="54" name="bGND_GNDA" color="1" fill="9" visible="yes" active="no"/>
-<layer number="56" name="wert" color="7" fill="1" visible="yes" active="no"/>
-<layer number="57" name="tCAD" color="7" fill="1" visible="yes" active="no"/>
+<layer number="46" name="Milling" color="3" fill="1" visible="no" active="no"/>
+<layer number="47" name="Measures" color="7" fill="1" visible="no" active="no"/>
+<layer number="48" name="Document" color="7" fill="1" visible="no" active="no"/>
+<layer number="49" name="Reference" color="7" fill="1" visible="no" active="no"/>
+<layer number="50" name="dxf" color="7" fill="1" visible="no" active="no"/>
+<layer number="51" name="tDocu" color="7" fill="1" visible="no" active="no"/>
+<layer number="52" name="bDocu" color="7" fill="1" visible="no" active="no"/>
+<layer number="53" name="tGND_GNDA" color="7" fill="9" visible="no" active="no"/>
+<layer number="54" name="bGND_GNDA" color="1" fill="9" visible="no" active="no"/>
+<layer number="56" name="wert" color="7" fill="1" visible="no" active="no"/>
+<layer number="57" name="tCAD" color="7" fill="1" visible="no" active="no"/>
 <layer number="90" name="Modules" color="5" fill="1" visible="yes" active="yes"/>
 <layer number="91" name="Nets" color="2" fill="1" visible="yes" active="yes"/>
@@
 <part name="P+12" library="supply1" deviceset="+5V" device=""/>
 <part name="C4P" library="rcl" deviceset="C-EU" device="C0805" value="100n"/>
-<part name="R_R" library="resistor" deviceset="R-TRIMM" device="3296W"/>
-<part name="R_G" library="resistor" deviceset="R-TRIMM" device="3296W"/>
-<part name="R_B" library="resistor" deviceset="R-TRIMM" device="3296W"/>
+<part name="R_R" library="Speccy" deviceset="R-TRIMM" device="3296W"/>
+<part name="R_G" library="Speccy" deviceset="R-TRIMM" device="3296W"/>
+<part name="R_B" library="Speccy" deviceset="R-TRIMM" device="3296W"/>
 <part name="GND16" library="supply1" deviceset="GND" device=""/>
 <part name="C2P" library="rcl" deviceset="C-EU" device="C0805" value="100n"/>
 <part name="C3P" library="rcl" deviceset="C-EU" device="C0805" value="100n"/>
 <part name="C1P" library="rcl" deviceset="C-EU" device="C0805" value="100n"/>
-<part name="R_SY" library="resistor" deviceset="R-TRIMM" device="3296W"/>
+<part name="R_SY" library="Speccy" deviceset="R-TRIMM" device="3296W"/>
 <part name="R9P" library="rcl" deviceset="R-EU_" device="R1206" value="75"/>
 <part name="C9P" library="rcl" deviceset="CPOL-EU" device="E2.5-5" value="220mf"/>

Commit message: .
Parts:
- added DD12: 74HCT04N, 74xx-eu:74HCT04N
- DD2: device altera_pga84:EPM7128-J84 -> Speccy:EPM7128-J84
Changed lines of the file:
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@@
 </classes>
 <parts>
-<part name="DD2" library="altera_pga84" deviceset="EPM7128-J84" device=""/>
+<part name="DD2" library="Speccy" deviceset="EPM7128-J84" device=""/>
 <part name="DD6" library="memory-hitachi" deviceset="62256P" device="" value="62256">
 <attribute name="MPN" value=""/>
@@
 <part name="R9P1" library="rcl" deviceset="R-EU_" device="R1206" value="75"/>
 <part name="R9P2" library="rcl" deviceset="R-EU_" device="R1206" value="75"/>
+<part name="DD12" library="74xx-eu" deviceset="74*04" device="N" technology="HCT"/>
 </parts>
 <sheets>
@@
 <attribute name="VALUE" x="372.11" y="74.422" size="1.778" layer="96" rot="R180"/>
 </instance>
+<instance part="DD12" gate="B" x="66.04" y="-25.4"/>
 </instances>
 <busses>

Commit message: .
Parts:
- removed DD12: 74HCT04N, 74xx-eu:74HCT04N
- DD11: value 74HCT04N -> 74LS04N; device 74xx-eu:74HCT04N -> Speccy:74LS04N
Connections:
- net +5V: now also DD11.7.VCC, DD2.2.VCC, DD2.3.VCC, DD2.4.VCCIO, DD2.5.VCCIO, DD2.6.VCCIO, DD2.7.VCCIO, DD2.8.VCCIO, DD2.9.VCCIO; no longer DD11P.VCC, DD21.VCC, DD22.VCC, DD23.VCCIO, DD24.VCCIO, DD25.VCCIO, DD26.VCCIO, DD27.VCCIO, DD28.VCCIO
- net A14: now also DD2.1.IO46; no longer DD2_.IO46
- net A15: now also DD2.1.IO45; no longer DD2_.IO45
- net AVR_INT: now also DD2.1.IO8; no longer DD2_.IO8
- net AVR_NOINT: now also DD2.1.IO13; no longer DD2_.IO13
- net AVR_PROM: now also DD2.1.OE2-GCLK2; no longer DD2_.OE2-GCLK2
- net AVR_TRDOS: now also DD2.1.IO123; no longer DD2_.IO123
- net AVR_WAIT: now also DD2.1.IO29; no longer DD2_.IO29
- net AY_BC: now also DD2.1.IO128; no longer DD2_.IO128
- net AY_BDIR: now also DD2.1.IO126; no longer DD2_.IO126
- net AY_CLK: now also DD2.1.IO125; no longer DD2_.IO125
- net B: now also DD2.1.IO64; no longer DD2_.IO64
- net BB: now also DD2.1.IO40; no longer DD2_.IO40
- net BG: now also DD2.1.IO43; no longer DD2_.IO43
- net BR: now also DD2.1.IO38; no longer DD2_.IO38
- net CLK: now also DD11.3.O, DD2.1.GCLK1; no longer DD11C.O, DD2_.GCLK1
- net CLK_CPU: now also DD2.1.IO17; no longer DD2_.IO17
- net FC: now also DD11.6.O; no longer DD11D.O
- net G: now also DD2.1.IO61; no longer DD2_.IO61
- net GND: now also DD11.7.GND, DD2.10.GND, DD2.11.GND, DD2.12.GND, DD2.13.GND, DD2.14.GND, DD2.15.GND, DD2.16.GND, DD2.17.GND; no longer DD11P.GND, DD210.GND, DD211.GND, DD212.GND, DD213.GND, DD214.GND, DD215.GND, DD216.GND, DD29.GND
- net INT: now also DD2.1.IO19; no longer DD2_.IO19
- net IOREQ: now also DD2.1.IO21; no longer DD2_.IO21
- net M1: now also DD2.1.IO27; no longer DD2_.IO27
- net MREQ: now also DD2.1.IO24; no longer DD2_.IO24
- net N$1: now also DD11.2.O, DD11.3.I; no longer DD11B.O, DD11C.I
- net N$12: now also DD11.1.I; no longer DD11A.I
- net N$43: now also DD11.4.O, DD11.5.I; no longer DD11E.I, DD11F.O
- net N$44: now also DD11.5.O, DD11.6.I; no longer DD11D.I, DD11E.O
- net N$45: now also DD11.4.I; no longer DD11F.I
- net N$5: now also DD11.1.O, DD11.2.I; no longer DD11A.O, DD11B.I
- net R: now also DD2.1.IO37; no longer DD2_.IO37
- net RA14: now also DD2.1.IO118; no longer DD2_.IO118
- net RA15: now also DD2.1.IO117; no longer DD2_.IO117
- net RA16: now also DD2.1.IO115; no longer DD2_.IO115
- net RAM_CS: now also DD2.1.IO5; no longer DD2_.IO5
- net RD: now also DD2.1.IO16; no longer DD2_.IO16
- net ROM_A14: now also DD2.1.IO35; no longer DD2_.IO35
- net ROM_A15: now also DD2.1.IO56; no longer DD2_.IO56
- net ROM_CS: now also DD2.1.IO14; no longer DD2_.IO14
- net RST_CPU: now also DD2.1.GCLR/; no longer DD2_.GCLR/
- net SPEAKER: now also DD2.1.IO59; no longer DD2_.IO59
- net SYNC: now also DD2.1.IO57; no longer DD2_.IO57
- net TAPE_IN: now also DD2.1.IO3; no longer DD2_.IO3
- net TCK: now also DD2.1.TCK/IO96; no longer DD2_.TCK/IO96
- net TDI: now also DD2.1.IO32/TDI; no longer DD2_.IO32/TDI
- net TDO: now also DD2.1.TDO/IO112; no longer DD2_.TDO/IO112
- net TMS: now also DD2.1.IO48/TMS; no longer DD2_.IO48/TMS
- net VA0: now also DD2.1.IO86; no longer DD2_.IO86
- net VA1: now also DD2.1.IO80; no longer DD2_.IO80
- net VA10: now also DD2.1.IO77; no longer DD2_.IO77
- net VA11: now also DD2.1.IO85; no longer DD2_.IO85
- net VA12: now also DD2.1.IO88; no longer DD2_.IO88
- net VA13: now also DD2.1.IO93; no longer DD2_.IO93
- net VA14: now also DD2.1.IO120; no longer DD2_.IO120
- net VA2: now also DD2.1.IO75; no longer DD2_.IO75
- net VA3: now also DD2.1.IO72; no longer DD2_.IO72
- net VA4: now also DD2.1.IO67; no longer DD2_.IO67
- net VA5: now also DD2.1.IO51; no longer DD2_.IO51
- net VA6: now also DD2.1.IO53; no longer DD2_.IO53
- net VA7: now also DD2.1.IO65; no longer DD2_.IO65
- net VA8: now also DD2.1.IO69; no longer DD2_.IO69
- net VA9: now also DD2.1.IO73; no longer DD2_.IO73
- net VAGEN: now also DD2.1.IO6; no longer DD2_.IO6
- net VD0: now also DD2.1.IO105; no longer DD2_.IO105
- net VD1: now also DD2.1.IO107; no longer DD2_.IO107
- net VD2: now also DD2.1.IO109; no longer DD2_.IO109
- net VD3: now also DD2.1.IO94; no longer DD2_.IO94
- net VD4: now also DD2.1.IO97; no longer DD2_.IO97
- net VD5: now also DD2.1.IO99; no longer DD2_.IO99
- net VD6: now also DD2.1.IO101; no longer DD2_.IO101
- net VD7: now also DD2.1.IO104; no longer DD2_.IO104
- net VRAM: now also DD2.1.IO91; no longer DD2_.IO91
- net VRD: now also DD2.1.IO83; no longer DD2_.IO83
- net VWR: now also DD2.1.IO49; no longer DD2_.IO49
- net WAIT_CPU: now also DD2.1.IO25; no longer DD2_.IO25
- net WR: now also DD2.1.IO11; no longer DD2_.IO11
