File: Speccy2007_128K_Ljubitel.sch (EAGLE design)
At the start: 103 parts, among them IC1 74HC74N, X2 SCART-F, X5 ByteBlaster, X6 AVRISP

Commit message: .
Parts:
- removed DA2: CXA1645, cxa1645:CXA1645-P
- removed IC1: 74HC74N, 74xx-eu:74HC74N
- added DD12: 74HC74N, 74xx-eu:74HC74N
- R12: device rcl:R-EU_R0805 -> rcl:R-EU_R1206
- R24: device rcl:R-EU_R1206 -> Speccy:R-EU_0207/10
- R7: device rcl:R-EU_0207/10 -> Speccy:R-EU_0207/10
- renumbered C2HC to CRL

Commit message: .
Parts:
- added R3: 1k, rcl:R-EU_R0805
Connections:
- new net N$38: DD12A.!Q, DD12A.D
- new net N$40: DD12A.CLR, DD12A.PRE, DD12B.CLR, DD12B.PRE, R3.1
- new net N$48: DD12B.!Q, DD12B.D
- net +5V: now also R3.2
- net FC: now also DD12A.CLK
Other:
- moved on the sheet: DD12A
Changed lines of the file:
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@@
 <part name="DD12" library="74xx-eu" deviceset="74*74" device="N" technology="HC"/>
 <part name="Q1" library="crystal" deviceset="CRYSTAL" device="HC49U-H"/>
+<part name="P+15" library="supply1" deviceset="+5V" device=""/>
+<part name="R3" library="rcl" deviceset="R-EU_" device="R0805" value="1k"/>
 </parts>
 <sheets>
@@
 <instance part="R1" gate="G$1" x="106.68" y="7.62"/>
 <instance part="R2" gate="G$1" x="129.54" y="226.06"/>
-<instance part="DD12" gate="A" x="190.5" y="233.68"/>
+<instance part="DD12" gate="A" x="342.9" y="25.4"/>
 <instance part="Q1" gate="G$1" x="76.2" y="2.54"/>
+<instance part="P+15" gate="1" x="320.04" y="48.26" smashed="yes" rot="MR0">
+<attribute name="VALUE" x="317.5" y="50.8" size="1.778" layer="96" rot="MR180"/>
+</instance>
+<instance part="R3" gate="G$1" x="325.12" y="38.1" smashed="yes" rot="R90">
+<attribute name="NAME" x="323.85" y="41.6814" size="1.778" layer="95" rot="R180"/>
+<attribute name="VALUE" x="323.85" y="38.862" size="1.778" layer="96" rot="R180"/>
+</instance>
+<instance part="DD12" gate="B" x="342.9" y="2.54"/>
 </instances>
 <busses>
@@
 <junction x="60.96" y="238.76"/>
 </segment>
+<segment>
+<pinref part="R3" gate="G$1" pin="2"/>
+<pinref part="P+15" gate="1" pin="+5V"/>
+<wire x1="325.12" y1="43.18" x2="320.04" y2="45.72" width="0.1524" layer="91"/>
+</segment>
 </net>
 <net name="A0" class="0">
@@
 <wire x1="307.34" y1="30.48" x2="312.42" y2="30.48" width="0.1524" layer="91"/>
 <label x="307.34" y="30.48" size="1.778" layer="95"/>
+<junction x="312.42" y="30.48"/>
+<pinref part="DD12" gate="A" pin="CLK"/>
+<wire x1="330.2" y1="22.86" x2="317.5" y2="22.86" width="0.1524" layer="91"/>
+<wire x1="317.5" y1="22.86" x2="317.5" y2="30.48" width="0.1524" layer="91"/>
+<wire x1="317.5" y1="30.48" x2="312.42" y2="30.48" width="0.1524" layer="91"/>
 </segment>
 <segment>
@@
 </segment>
 </net>
+<net name="N$38" class="0">
+<segment>
+<pinref part="DD12" gate="A" pin="D"/>
+<wire x1="330.2" y1="27.94" x2="327.66" y2="27.94" width="0.1524" layer="91"/>
+<wire x1="327.66" y1="27.94" x2="327.66" y2="38.1" width="0.1524" layer="91"/>
+<wire x1="327.66" y1="38.1" x2="358.14" y2="38.1" width="0.1524" layer="91"/>
+<wire x1="358.14" y1="38.1" x2="358.14" y2="20.32" width="0.1524" layer="91"/>
+<pinref part="DD12" gate="A" pin="!Q"/>
+<wire x1="358.14" y1="20.32" x2="355.6" y2="20.32" width="0.1524" layer="91"/>
+</segment>
+</net>
+<net name="N$40" class="0">
+<segment>
+<pinref part="DD12" gate="A" pin="CLR"/>
+<wire x1="330.2" y1="20.32" x2="325.12" y2="20.32" width="0.1524" layer="91"/>
+<wire x1="325.12" y1="20.32" x2="325.12" y2="30.48" width="0.1524" layer="91"/>
+<pinref part="DD12" gate="A" pin="PRE"/>
+<wire x1="325.12" y1="30.48" x2="330.2" y2="30.48" width="0.1524" layer="91"/>
+<wire x1="325.12" y1="30.48" x2="325.12" y2="33.02" width="0.1524" layer="91"/>
+<junction x="325.12" y="30.48"/>
+<pinref part="R3" gate="G$1" pin="1"/>
+<pinref part="DD12" gate="B" pin="PRE"/>
+<wire x1="330.2" y1="7.62" x2="325.12" y2="7.62" width="0.1524" layer="91"/>
+<wire x1="325.12" y1="7.62" x2="325.12" y2="20.32" width="0.1524" layer="91"/>
+<pinref part="DD12" gate="B" pin="CLR"/>
+<wire x1="330.2" y1="-2.54" x2="325.12" y2="-2.54" width="0.1524" layer="91"/>
+<wire x1="325.12" y1="-2.54" x2="325.12" y2="7.62" width="0.1524" layer="91"/>
+</segment>
+</net>
+<net name="N$48" class="0">
+<segment>
+<pinref part="DD12" gate="B" pin="D"/>
+<wire x1="330.2" y1="5.08" x2="327.66" y2="5.08" width="0.1524" layer="91"/>
+<wire x1="327.66" y1="5.08" x2="327.66" y2="12.7" width="0.1524" layer="91"/>
+<wire x1="327.66" y1="12.7" x2="358.14" y2="12.7" width="0.1524" layer="91"/>
+<wire x1="358.14" y1="12.7" x2="358.14" y2="-2.54" width="0.1524" layer="91"/>
+<pinref part="DD12" gate="B" pin="!Q"/>
+<wire x1="358.14" y1="-2.54" x2="355.6" y2="-2.54" width="0.1524" layer="91"/>
+</segment>
+</net>

Commit message: head
Parts:
- added IC1: 74AC74D, 74xx-eu:74AC74D
- added IC2: AP1117, AWJLEagleLib:AP1117
Connections:
- net +3V3: now also IC2.OUT, IC2.OUT'
- net +5V: now also IC2.IN
- net GND: now also IC2.GND
Changed lines of the file:
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@@
 <grid distance="100" unitdist="mil" unit="mil" style="lines" multiple="1" display="yes" altdistance="0.01" altunitdist="inch" altunit="inch"/>
 <layers>
-<layer number="1" name="Top" color="4" fill="1" visible="yes" active="no"/>
-<layer number="2" name="Route2" color="1" fill="3" visible="yes" active="no"/>
-<layer number="3" name="Route3" color="4" fill="3" visible="yes" active="no"/>
-<layer number="4" name="Route4" color="1" fill="4" visible="yes" active="no"/>
-<layer number="5" name="Route5" color="4" fill="4" visible="yes" active="no"/>
-<layer number="6" name="Route6" color="1" fill="8" visible="yes" active="no"/>
-<layer number="7" name="Route7" color="4" fill="8" visible="yes" active="no"/>
-<layer number="8" name="Route8" color="1" fill="2" visible="yes" active="no"/>
-<layer number="9" name="Route9" color="4" fill="2" visible="yes" active="no"/>
-<layer number="10" name="Route10" color="1" fill="7" visible="yes" active="no"/>
-<layer number="11" name="Route11" color="4" fill="7" visible="yes" active="no"/>
-<layer number="12" name="Route12" color="1" fill="5" visible="yes" active="no"/>
-<layer number="13" name="Route13" color="4" fill="5" visible="yes" active="no"/>
-<layer number="14" name="Route14" color="1" fill="6" visible="yes" active="no"/>
-<layer number="15" name="Route15" color="4" fill="6" visible="yes" active="no"/>
-<layer number="16" name="Bottom" color="1" fill="1" visible="yes" active="no"/>
-<layer number="17" name="Pads" color="2" fill="1" visible="yes" active="no"/>
-<layer number="18" name="Vias" color="2" fill="1" visible="yes" active="no"/>
-<layer number="19" name="Unrouted" color="6" fill="1" visible="yes" active="no"/>
-<layer number="20" name="Dimension" color="15" fill="1" visible="yes" active="no"/>
-<layer number="21" name="tPlace" color="7" fill="1" visible="yes" active="no"/>
-<layer number="22" name="bPlace" color="7" fill="1" visible="yes" active="no"/>
-<layer number="23" name="tOrigins" color="15" fill="1" visible="yes" active="no"/>
-<layer number="24" name="bOrigins" color="15" fill="1" visible="yes" active="no"/>
-<layer number="25" name="tNames" color="7" fill="1" visible="yes" active="no"/>
-<layer number="26" name="bNames" color="7" fill="1" visible="yes" active="no"/>
-<layer number="27" name="tValues" color="7" fill="1" visible="yes" active="no"/>
-<layer number="28" name="bValues" color="7" fill="1" visible="yes" active="no"/>
+<layer number="1" name="Top" color="4" fill="1" visible="no" active="no"/>
+<layer number="2" name="Route2" color="1" fill="3" visible="no" active="no"/>
+<layer number="3" name="Route3" color="4" fill="3" visible="no" active="no"/>
+<layer number="4" name="Route4" color="1" fill="4" visible="no" active="no"/>
+<layer number="5" name="Route5" color="4" fill="4" visible="no" active="no"/>
+<layer number="6" name="Route6" color="1" fill="8" visible="no" active="no"/>
+<layer number="7" name="Route7" color="4" fill="8" visible="no" active="no"/>
+<layer number="8" name="Route8" color="1" fill="2" visible="no" active="no"/>
+<layer number="9" name="Route9" color="4" fill="2" visible="no" active="no"/>
+<layer number="10" name="Route10" color="1" fill="7" visible="no" active="no"/>
+<layer number="11" name="Route11" color="4" fill="7" visible="no" active="no"/>
+<layer number="12" name="Route12" color="1" fill="5" visible="no" active="no"/>
+<layer number="13" name="Route13" color="4" fill="5" visible="no" active="no"/>
+<layer number="14" name="Route14" color="1" fill="6" visible="no" active="no"/>
+<layer number="15" name="Route15" color="4" fill="6" visible="no" active="no"/>
+<layer number="16" name="Bottom" color="1" fill="1" visible="no" active="no"/>
+<layer number="17" name="Pads" color="2" fill="1" visible="no" active="no"/>
+<layer number="18" name="Vias" color="2" fill="1" visible="no" active="no"/>
+<layer number="19" name="Unrouted" color="6" fill="1" visible="no" active="no"/>
+<layer number="20" name="Dimension" color="15" fill="1" visible="no" active="no"/>
+<layer number="21" name="tPlace" color="7" fill="1" visible="no" active="no"/>
+<layer number="22" name="bPlace" color="7" fill="1" visible="no" active="no"/>
+<layer number="23" name="tOrigins" color="15" fill="1" visible="no" active="no"/>
+<layer number="24" name="bOrigins" color="15" fill="1" visible="no" active="no"/>
+<layer number="25" name="tNames" color="7" fill="1" visible="no" active="no"/>
+<layer number="26" name="bNames" color="7" fill="1" visible="no" active="no"/>
+<layer number="27" name="tValues" color="7" fill="1" visible="no" active="no"/>
+<layer number="28" name="bValues" color="7" fill="1" visible="no" active="no"/>
 <layer number="29" name="tStop" color="7" fill="3" visible="no" active="no"/>
 <layer number="30" name="bStop" color="7" fill="6" visible="no" active="no"/>
@@
 <layer number="35" name="tGlue" color="7" fill="4" visible="no" active="no"/>
 <layer number="36" name="bGlue" color="7" fill="5" visible="no" active="no"/>
-<layer number="37" name="tTest" color="7" fill="1" visible="yes" active="no"/>
-<layer number="38" name="bTest" color="7" fill="1" visible="yes" active="no"/>
+<layer number="37" name="tTest" color="7" fill="1" visible="no" active="no"/>
+<layer number="38" name="bTest" color="7" fill="1" visible="no" active="no"/>
 <layer number="39" name="tKeepout" color="4" fill="11" visible="no" active="no"/>
 <layer number="40" name="bKeepout" color="1" fill="11" visible="no" active="no"/>
@@
 <layer number="44" name="Drills" color="7" fill="1" visible="no" active="no"/>
 <layer number="45" name="Holes" color="7" fill="1" visible="no" active="no"/>
-<layer number="46" name="Milling" color="3" fill="1" visible="yes" active="no"/>
-<layer number="47" name="Measures" color="7" fill="1" visible="yes" active="no"/>
-<layer number="48" name="Document" color="7" fill="1" visible="yes" active="no"/>
-<layer number="49" name="Reference" color="7" fill="1" visible="yes" active="no"/>
-<layer number="50" name="dxf" color="7" fill="1" visible="yes" active="no"/>
-<layer number="51" name="tDocu" color="7" fill="1" visible="yes" active="no"/>
-<layer number="52" name="bDocu" color="7" fill="1" visible="yes" active="no"/>
-<layer number="53" name="tGND_GNDA" color="7" fill="9" visible="yes" active="no"/>
-<layer number="54" name="bGND_GNDA" color="1" fill="9" visible="yes" active="no"/>
-<layer number="56" name="wert" color="7" fill="1" visible="yes" active="no"/>
-<layer number="57" name="tCAD" color="7" fill="1" visible="yes" active="no"/>
+<layer number="46" name="Milling" color="3" fill="1" visible="no" active="no"/>
+<layer number="47" name="Measures" color="7" fill="1" visible="no" active="no"/>
+<layer number="48" name="Document" color="7" fill="1" visible="no" active="no"/>
+<layer number="49" name="Reference" color="7" fill="1" visible="no" active="no"/>
+<layer number="50" name="dxf" color="7" fill="1" visible="no" active="no"/>
+<layer number="51" name="tDocu" color="7" fill="1" visible="no" active="no"/>
+<layer number="52" name="bDocu" color="7" fill="1" visible="no" active="no"/>
+<layer number="53" name="tGND_GNDA" color="7" fill="9" visible="no" active="no"/>
+<layer number="54" name="bGND_GNDA" color="1" fill="9" visible="no" active="no"/>
+<layer number="56" name="wert" color="7" fill="1" visible="no" active="no"/>
+<layer number="57" name="tCAD" color="7" fill="1" visible="no" active="no"/>
 <layer number="90" name="Modules" color="5" fill="1" visible="yes" active="yes"/>
 <layer number="91" name="Nets" color="2" fill="1" visible="yes" active="yes"/>
@@
 <part name="P+15" library="supply1" deviceset="+5V" device=""/>
 <part name="R3" library="rcl" deviceset="R-EU_" device="R0805" value="1k"/>
+<part name="IC2" library="AWJLEagleLib" deviceset="AP1117" device=""/>
+<part name="GND25" library="supply1" deviceset="GND" device=""/>
+<part name="P+16" library="supply1" deviceset="+5V" device=""/>
+<part name="IC1" library="74xx-eu" deviceset="74*74" device="D" technology="AC"/>
 </parts>
 <sheets>
@@
 </instance>
 <instance part="DD12" gate="B" x="342.9" y="2.54"/>
+<instance part="IC2" gate="G$1" x="368.3" y="147.32" smashed="yes">
+<attribute name="NAME" x="355.6" y="142.24" size="1.778" layer="95"/>
+<attribute name="VALUE" x="355.6" y="139.7" size="1.778" layer="96"/>
+</instance>
+<instance part="GND25" gate="1" x="368.3" y="134.62" rot="MR0"/>
+<instance part="P+16" gate="1" x="355.6" y="152.4" smashed="yes" rot="MR0">
+<attribute name="VALUE" x="353.06" y="154.94" size="1.778" layer="96" rot="MR180"/>
+</instance>
+<instance part="IC1" gate="A" x="292.1" y="-5.08"/>
 </instances>
 <busses>
@@
 <wire x1="386.08" y1="137.16" x2="386.08" y2="134.62" width="0.1524" layer="91"/>
 </segment>
+<segment>
+<pinref part="IC2" gate="G$1" pin="GND"/>
+<pinref part="GND25" gate="1" pin="GND"/>
+<wire x1="368.3" y1="139.7" x2="368.3" y2="137.16" width="0.1524" layer="91"/>
+</segment>
 </net>
 <net name="+5V" class="0">
@@
 <wire x1="325.12" y1="43.18" x2="320.04" y2="45.72" width="0.1524" layer="91"/>
 </segment>
+<segment>
+<pinref part="IC2" gate="G$1" pin="IN"/>
+<wire x1="360.68" y1="147.32" x2="355.6" y2="147.32" width="0.1524" layer="91"/>
+<pinref part="P+16" gate="1" pin="+5V"/>
+<wire x1="355.6" y1="147.32" x2="355.6" y2="149.86" width="0.1524" layer="91"/>
+</segment>
 </net>
 <net name="A0" class="0">
@@
 <wire x1="386.08" y1="149.86" x2="386.08" y2="147.32" width="0.1524" layer="91"/>
 <junction x="386.08" y="147.32"/>
+<wire x1="375.92" y1="147.32" x2="378.46" y2="147.32" width="0.1524" layer="91"/>
+<pinref part="IC2" gate="G$1" pin="OUT"/>
+<wire x1="378.46" y1="147.32" x2="386.08" y2="147.32" width="0.1524" layer="91"/>
+<wire x1="378.46" y1="147.32" x2="378.46" y2="144.78" width="0.1524" layer="91"/>
+<pinref part="IC2" gate="G$1" pin="OUT'"/>
+<wire x1="378.46" y1="144.78" x2="375.92" y2="144.78" width="0.1524" layer="91"/>
+<junction x="378.46" y="147.32"/>
 </segment>
 </net>

Commit message: .
Parts:
- removed IC1: 74AC74D, 74xx-eu:74AC74D
- added CT: 100n, rcl:C-EUC1206
- added EXTPOWER: POWERSUPPLY_DC21MMX, SmartPrj:POWERSUPPLY_DC21MMX
- C1Y, C2Y: device rcl:CPOL-EUE2.5-6 -> rcl:CPOL-EUE2.5-5
- DD12: value 74HC74N -> 74LS74O; device 74xx-eu:74HC74N -> Speccy:74LS74O
- R8P: device rcl:R-EU_M0805 -> rcl:R-EU_R1206
- renumbered IC2 to DA2
Connections:
- removed net N$38 (its old number): DD12A.!Q, DD12A.D
- new net FCI: DD11.6.O, DD12B.CLK
- net +5V: now also CT.1, DD12P.VCC, EXTPOWER.2
- net FC: now also DD12B.Q; no longer DD11.6.O, DD12A.CLK
- net GND: now also CT.2, DD12P.GND, EXTPOWER.1, EXTPOWER.3
- net N$40: now also DD12A.CLK, DD12A.D
Other:
- moved on the sheet: DD12A, DD12B, R3

Commit message: .
Parts:
- removed EXTPOWER: POWERSUPPLY_DC21MMX, SmartPrj:POWERSUPPLY_DC21MMX
- added Q2: (no value), crystal:CRYSTALHC49U-H
- added X1: 5V, Speccy:POWER3.5
- X3: value MINI-DIN6PTH -> PS/2 KB
- X5: device con-lstb:MA05-2 -> Speccy:MA05-2
- X6: device con-lstb:MA03-2 -> Speccy:MA03-2
- renumbered J1 to X4, PS2KB to X3
Connections:
- net +5V: now also X1.1; no longer EXTPOWER.2
- net GND: now also X1.2, X1.3; no longer EXTPOWER.1, EXTPOWER.3
