File: Speccy2007_128K_Ljubitel.sch (EAGLE design)
At the start: 107 parts, among them X1 5V, X2 SCART-F, X3 PS/2 KB, X5 ByteBlaster, X6 AVRISP

Commit message: .
Parts:
- removed Q1, Q2: (no value), crystal:CRYSTALHC49U-H
- C1Y, C2Y, C6P, C8P, C8P1, C8P2, C9, C9P: device rcl:CPOL-EUE2.5-5 -> Speccy:CPOL-EUE2.5-5
- Z1, Z2: device special:XTAL/S -> Speccy:CRYSTALHC49U-H
Connections:
- net N$44: now also Z2.2; no longer Z2.1
- net N$45: now also Z2.1; no longer Z2.2
Changed lines of the file:
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@@
 <part name="GND1" library="supply1" deviceset="GND" device=""/>
 <part name="P+2" library="supply1" deviceset="+5V" device=""/>
-<part name="Z1" library="special" deviceset="XTAL/S" device="" value="14Mhz"/>
+<part name="Z1" library="Speccy" deviceset="CRYSTAL" device="HC49U-H" value="14Mhz"/>
 <part name="R34" library="rcl" deviceset="R-EU_" device="R0805" value="360"/>
 <part name="P+3" library="supply1" deviceset="+5V" device=""/>
@@
 <part name="R7Y" library="rcl" deviceset="R-EU_" device="R0805" value="4k7"/>
 <part name="C3Y" library="rcl" deviceset="C-EU" device="C0805" value="0.1"/>
-<part name="C1Y" library="rcl" deviceset="CPOL-EU" device="E2.5-5" value="1m"/>
+<part name="C1Y" library="Speccy" deviceset="CPOL-EU" device="E2.5-5" value="1m"/>
 <part name="R5Y" library="rcl" deviceset="R-EU_" device="R1206" value="5k1"/>
 <part name="GND8" library="supply1" deviceset="GND" device=""/>
-<part name="C2Y" library="rcl" deviceset="CPOL-EU" device="E2.5-5" value="1m"/>
+<part name="C2Y" library="Speccy" deviceset="CPOL-EU" device="E2.5-5" value="1m"/>
 <part name="R8Y" library="rcl" deviceset="R-EU_" device="R0805" value="5k1"/>
 <part name="R9Y" library="rcl" deviceset="R-EU_" device="R0805" value="4k7"/>
@@
 <part name="DD11" library="Speccy" deviceset="74*04" device="N" technology="LS" value="74LS04N"/>
 <part name="-R3" library="rcl" deviceset="R-EU_" device="R0805" value="360"/>
-<part name="Z2" library="special" deviceset="XTAL/S" device="" value="4.43Mhz"/>
+<part name="Z2" library="Speccy" deviceset="CRYSTAL" device="HC49U-H" value="4.43Mhz"/>
 <part name="R112" library="rcl" deviceset="R-EU_" device="R0805" value="360"/>
 <part name="R1223" library="rcl" deviceset="R-EU_" device="R0805" value="360"/>
@@
 <part name="R_SY" library="Speccy" deviceset="R-TRIMM" device="3296W"/>
 <part name="R9P" library="rcl" deviceset="R-EU_" device="R1206" value="75"/>
-<part name="C9P" library="rcl" deviceset="CPOL-EU" device="E2.5-5" value="220mf"/>
+<part name="C9P" library="Speccy" deviceset="CPOL-EU" device="E2.5-5" value="220mf"/>
 <part name="R5P" library="rcl" deviceset="R-EU_" device="M1206" value="16k*"/>
 <part name="C5P" library="rcl" deviceset="C-EU" device="C1206" value="100n"/>
 <part name="R6P" library="rcl" deviceset="R-EU_" device="R1206" value="47k"/>
-<part name="C6P" library="rcl" deviceset="CPOL-EU" device="E2.5-5" value="10mf"/>
+<part name="C6P" library="Speccy" deviceset="CPOL-EU" device="E2.5-5" value="10mf"/>
 <part name="R8P" library="rcl" deviceset="R-EU_" device="R1206" value="75"/>
-<part name="C8P" library="rcl" deviceset="CPOL-EU" device="E2.5-5" value="220mf"/>
+<part name="C8P" library="Speccy" deviceset="CPOL-EU" device="E2.5-5" value="220mf"/>
 <part name="R1D" library="rcl" deviceset="R-EU_" device="R0805" value="10k"/>
 <part name="R2D" library="rcl" deviceset="R-EU_" device="M0805" value="10k"/>
@@
 <part name="C8" library="rcl" deviceset="C-EU" device="C0805" value="100n"/>
 <part name="GND23" library="supply1" deviceset="GND" device=""/>
-<part name="C9" library="rcl" deviceset="CPOL-EU" device="E2.5-5" value="220mf"/>
+<part name="C9" library="Speccy" deviceset="CPOL-EU" device="E2.5-5" value="220mf"/>
 <part name="GND24" library="supply1" deviceset="GND" device=""/>
 <part name="P+4" library="supply1" deviceset="+5V" device=""/>
@@
 <part name="+3V1" library="supply1" deviceset="+3V3" device=""/>
 <part name="+3V2" library="supply1" deviceset="+3V3" device=""/>
-<part name="C8P1" library="rcl" deviceset="CPOL-EU" device="E2.5-5" value="220mf"/>
-<part name="C8P2" library="rcl" deviceset="CPOL-EU" device="E2.5-5" value="220mf"/>
+<part name="C8P1" library="Speccy" deviceset="CPOL-EU" device="E2.5-5" value="220mf"/>
+<part name="C8P2" library="Speccy" deviceset="CPOL-EU" device="E2.5-5" value="220mf"/>
 <part name="R9P1" library="rcl" deviceset="R-EU_" device="R1206" value="75"/>
 <part name="R9P2" library="rcl" deviceset="R-EU_" device="R1206" value="75"/>
@@
 <part name="R2" library="rcl" deviceset="R-EU_" device="M1206"/>
 <part name="DD12" library="Speccy" deviceset="74*74" device="O" technology="LS" value="74LS74O"/>
-<part name="Q1" library="crystal" deviceset="CRYSTAL" device="HC49U-H"/>
 <part name="P+15" library="supply1" deviceset="+5V" device=""/>
 <part name="R3" library="rcl" deviceset="R-EU_" device="R0805" value="1k"/>
@@
 <part name="GND26" library="supply1" deviceset="GND" device=""/>
 <part name="CT" library="rcl" deviceset="C-EU" device="C1206" value="100n"/>
-<part name="Q2" library="crystal" deviceset="CRYSTAL" device="HC49U-H">
-<attribute name="MF" value=""/>
-<attribute name="MPN" value=""/>
-<attribute name="OC_FARNELL" value="1666973"/>
-<attribute name="OC_NEWARK" value="unknown"/>
-</part>
 <part name="X1" library="Speccy" deviceset="POWER3.5" device="" value="5V"/>
 <part name="GND28" library="supply1" deviceset="GND" device=""/>
@@
 <instance part="DD11" gate=".4" x="246.38" y="30.48"/>
 <instance part="-R3" gate="G$1" x="243.84" y="20.32"/>
-<instance part="Z2" gate="G$1" x="259.08" y="40.64" smashed="yes" rot="R180">
-<attribute name="NAME" x="250.19" y="43.18" size="1.778" layer="95" rot="R180"/>
-<attribute name="VALUE" x="254" y="39.37" size="1.778" layer="96" rot="R180"/>
+<instance part="Z2" gate="G$1" x="259.08" y="40.64" smashed="yes" rot="MR180">
+<attribute name="NAME" x="267.97" y="43.18" size="1.778" layer="95" rot="MR180"/>
+<attribute name="VALUE" x="264.16" y="39.37" size="1.778" layer="96" rot="MR180"/>
 </instance>
 <instance part="DD11" gate=".7" x="109.22" y="68.58"/>
@@
 <instance part="R2" gate="G$1" x="129.54" y="226.06"/>
 <instance part="DD12" gate="B" x="350.52" y="15.24"/>
-<instance part="Q1" gate="G$1" x="76.2" y="2.54"/>
 <instance part="P+15" gate="1" x="332.74" y="40.64" smashed="yes" rot="MR0">
 <attribute name="VALUE" x="330.2" y="43.18" size="1.778" layer="96" rot="MR180"/>
@@
 <instance part="GND26" gate="1" x="325.12" y="15.24" rot="MR0"/>
 <instance part="CT" gate="G$1" x="81.28" y="233.68"/>
-<instance part="Q2" gate="G$1" x="86.36" y="-2.54"/>
 <instance part="X1" gate="G$1" x="279.4" y="-5.08"/>
 <instance part="GND28" gate="1" x="287.02" y="-12.7" rot="MR0"/>
@@
 <wire x1="12.7" y1="20.32" x2="12.7" y2="30.48" width="0.1524" layer="91"/>
 <pinref part="Z1" gate="G$1" pin="2"/>
-<wire x1="33.02" y1="30.48" x2="12.7" y2="30.48" width="0.1524" layer="91"/>
+<wire x1="35.56" y1="30.48" x2="12.7" y2="30.48" width="0.1524" layer="91"/>
 <junction x="12.7" y="20.32"/>
 </segment>
@@
 <segment>
 <pinref part="Z1" gate="G$1" pin="1"/>
-<wire x1="43.18" y1="30.48" x2="63.5" y2="30.48" width="0.1524" layer="91"/>
+<wire x1="40.64" y1="30.48" x2="63.5" y2="30.48" width="0.1524" layer="91"/>
 <wire x1="63.5" y1="30.48" x2="63.5" y2="20.32" width="0.1524" layer="91"/>
 <pinref part="DD11" gate=".2" pin="O"/>
@@
 <net name="N$44" class="0">
 <segment>
-<pinref part="Z2" gate="G$1" pin="1"/>
-<wire x1="264.16" y1="40.64" x2="284.48" y2="40.64" width="0.1524" layer="91"/>
 <pinref part="R1223" gate="G$1" pin="2"/>
 <wire x1="274.32" y1="20.32" x2="284.48" y2="20.32" width="0.1524" layer="91"/>
@@
 <wire x1="284.48" y1="30.48" x2="287.02" y2="30.48" width="0.1524" layer="91"/>
 <junction x="284.48" y="30.48"/>
+<pinref part="Z2" gate="G$1" pin="2"/>
+<wire x1="261.62" y1="40.64" x2="284.48" y2="40.64" width="0.1524" layer="91"/>
 </segment>
 </net>
@@
 <wire x1="233.68" y1="20.32" x2="238.76" y2="20.32" width="0.1524" layer="91"/>
 <wire x1="233.68" y1="20.32" x2="233.68" y2="30.48" width="0.1524" layer="91"/>
-<pinref part="Z2" gate="G$1" pin="2"/>
 <wire x1="233.68" y1="30.48" x2="233.68" y2="40.64" width="0.1524" layer="91"/>
-<wire x1="233.68" y1="40.64" x2="254" y2="40.64" width="0.1524" layer="91"/>
 <pinref part="DD11" gate=".4" pin="I"/>
 <wire x1="233.68" y1="30.48" x2="236.22" y2="30.48" width="0.1524" layer="91"/>
 <junction x="233.68" y="30.48"/>
+<pinref part="Z2" gate="G$1" pin="1"/>
+<wire x1="256.54" y1="40.64" x2="233.68" y2="40.64" width="0.1524" layer="91"/>
 </segment>
 </net>

Commit message: .
Parts:
- added LED1: sdcard, led:LEDSML0805
- added LED2: power, led:LEDSML0805
Connections:
- net N$1: now also Z1.2; no longer Z1.1
- net N$12: now also Z1.1; no longer Z1.2
- net N$44: now also Z2.1; no longer Z2.2
- net N$45: now also Z2.2; no longer Z2.1
Changed lines of the file:
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@@
 <part name="GND28" library="supply1" deviceset="GND" device=""/>
 <part name="P+18" library="supply1" deviceset="+5V" device=""/>
+<part name="LED1" library="led" deviceset="LED" device="SML0805" value="sdcard"/>
+<part name="LED2" library="led" deviceset="LED" device="SML0805" value="power"/>
 </parts>
 <sheets>
@@
 <instance part="GND1" gate="1" x="27.94" y="147.32" rot="R270"/>
 <instance part="P+2" gate="1" x="86.36" y="106.68"/>
-<instance part="Z1" gate="G$1" x="38.1" y="30.48" smashed="yes" rot="R180">
-<attribute name="NAME" x="29.21" y="31.75" size="1.778" layer="95"/>
-<attribute name="VALUE" x="26.67" y="27.94" size="1.778" layer="96"/>
+<instance part="Z1" gate="G$1" x="38.1" y="30.48" smashed="yes" rot="MR180">
+<attribute name="NAME" x="46.99" y="31.75" size="1.778" layer="95" rot="MR0"/>
+<attribute name="VALUE" x="49.53" y="27.94" size="1.778" layer="96" rot="MR0"/>
 </instance>
 <instance part="R34" gate="G$1" x="25.4" y="12.7"/>
@@
 <instance part="DD11" gate=".4" x="246.38" y="30.48"/>
 <instance part="-R3" gate="G$1" x="243.84" y="20.32"/>
-<instance part="Z2" gate="G$1" x="259.08" y="40.64" smashed="yes" rot="MR180">
-<attribute name="NAME" x="267.97" y="43.18" size="1.778" layer="95" rot="MR180"/>
-<attribute name="VALUE" x="264.16" y="39.37" size="1.778" layer="96" rot="MR180"/>
+<instance part="Z2" gate="G$1" x="259.08" y="40.64" smashed="yes" rot="R180">
+<attribute name="NAME" x="250.19" y="43.18" size="1.778" layer="95" rot="R180"/>
+<attribute name="VALUE" x="254" y="39.37" size="1.778" layer="96" rot="R180"/>
 </instance>
 <instance part="DD11" gate=".7" x="109.22" y="68.58"/>
@@
 <attribute name="VALUE" x="284.48" y="5.08" size="1.778" layer="96" rot="MR180"/>
 </instance>
+<instance part="LED1" gate="G$1" x="386.08" y="195.58" rot="R90"/>
+<instance part="LED2" gate="G$1" x="386.08" y="208.28" rot="R90"/>
 </instances>
 <busses>
@@
 <wire x1="12.7" y1="20.32" x2="15.24" y2="20.32" width="0.1524" layer="91"/>
 <wire x1="12.7" y1="20.32" x2="12.7" y2="30.48" width="0.1524" layer="91"/>
-<pinref part="Z1" gate="G$1" pin="2"/>
-<wire x1="35.56" y1="30.48" x2="12.7" y2="30.48" width="0.1524" layer="91"/>
 <junction x="12.7" y="20.32"/>
+<pinref part="Z1" gate="G$1" pin="1"/>
+<wire x1="12.7" y1="30.48" x2="35.56" y2="30.48" width="0.1524" layer="91"/>
 </segment>
 </net>
 <net name="N$1" class="0">
 <segment>
-<pinref part="Z1" gate="G$1" pin="1"/>
-<wire x1="40.64" y1="30.48" x2="63.5" y2="30.48" width="0.1524" layer="91"/>
 <wire x1="63.5" y1="30.48" x2="63.5" y2="20.32" width="0.1524" layer="91"/>
 <pinref part="DD11" gate=".2" pin="O"/>
@@
 <pinref part="R112" gate="G$1" pin="2"/>
 <wire x1="53.34" y1="12.7" x2="63.5" y2="12.7" width="0.1524" layer="91"/>
+<pinref part="Z1" gate="G$1" pin="2"/>
+<wire x1="40.64" y1="30.48" x2="63.5" y2="30.48" width="0.1524" layer="91"/>
 </segment>
 </net>
@@
 <wire x1="284.48" y1="30.48" x2="287.02" y2="30.48" width="0.1524" layer="91"/>
 <junction x="284.48" y="30.48"/>
-<pinref part="Z2" gate="G$1" pin="2"/>
+<pinref part="Z2" gate="G$1" pin="1"/>
 <wire x1="261.62" y1="40.64" x2="284.48" y2="40.64" width="0.1524" layer="91"/>
 </segment>
@@
 <wire x1="233.68" y1="30.48" x2="236.22" y2="30.48" width="0.1524" layer="91"/>
 <junction x="233.68" y="30.48"/>
-<pinref part="Z2" gate="G$1" pin="1"/>
-<wire x1="256.54" y1="40.64" x2="233.68" y2="40.64" width="0.1524" layer="91"/>
+<pinref part="Z2" gate="G$1" pin="2"/>
+<wire x1="233.68" y1="40.64" x2="256.54" y2="40.64" width="0.1524" layer="91"/>
 </segment>
 </net>

Commit message: .
Parts:
- added R25, R26: 1k, rcl:R-EU_R0805
Connections:
- new net N$39: LED2.C, R25.2
- new net N$41: LED1.C, R26.2
- net +3V3: now also LED1.A, LED2.A
- net GND: now also R25.1
- net N$16: now also R26.1
- net N$44: now also Z2.2; no longer Z2.1
- net N$45: now also Z2.1; no longer Z2.2
Other:
- moved on the sheet: CE1, CM16, CRL, CT, CW29, CY, CZ80, LED1, LED2, R2, R22, X1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
