File: Speccy2007_128K_Ljubitel.sch (EAGLE design)
At the start: 109 parts, among them X1 5V, X2 SCART-F, X3 PS/2 KB, X5 ByteBlaster, X6 AVRISP

Commit message: .
Parts:
- X3: device SparkFun-Connectors:MINI-DIN6PTH -> Speccy:MINI-DIN6PTH
- renumbered LED1 to HL2, LED2 to HL1
Connections:
- net GND: now also X3.7
Changed lines of the file:
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@@
 <part name="R5" library="rcl" deviceset="R-EU_" device="R0805" value="470"/>
 <part name="R8" library="rcl" deviceset="R-EU_" device="R0805" value="330"/>
-<part name="X3" library="SparkFun-Connectors" deviceset="MINI-DIN6" device="PTH" value="PS/2 KB"/>
+<part name="X3" library="Speccy" deviceset="MINI-DIN6" device="PTH" value="PS/2 KB"/>
 <part name="DD3" library="Speccy" deviceset="621024" device="P" value="621024"/>
 <part name="P+11" library="supply1" deviceset="+5V" device=""/>
@@
 <part name="GND28" library="supply1" deviceset="GND" device=""/>
 <part name="P+18" library="supply1" deviceset="+5V" device=""/>
-<part name="LED1" library="led" deviceset="LED" device="SML0805" value="sdcard"/>
-<part name="LED2" library="led" deviceset="LED" device="SML0805" value="power"/>
+<part name="HL2" library="led" deviceset="LED" device="SML0805" value="sdcard"/>
+<part name="HL1" library="led" deviceset="LED" device="SML0805" value="power"/>
 <part name="R25" library="rcl" deviceset="R-EU_" device="R0805" value="1k"/>
 <part name="GND27" library="supply1" deviceset="GND" device=""/>
@@
 <instance part="X3" gate="G$1" x="261.62" y="231.14" smashed="yes" rot="MR0">
 <attribute name="VALUE" x="269.24" y="220.98" size="1.778" layer="96" rot="MR0"/>
-<attribute name="NAME" x="264.16" y="242.062" size="1.778" layer="95" rot="MR0"/>
+<attribute name="NAME" x="264.16" y="244.602" size="1.778" layer="95" rot="MR0"/>
 </instance>
 <instance part="DD3" gate="G$1" x="175.26" y="175.26"/>
@@
 <attribute name="VALUE" x="27.94" y="236.22" size="1.778" layer="96" rot="MR180"/>
 </instance>
-<instance part="LED1" gate="G$1" x="370.84" y="198.12" rot="R90"/>
-<instance part="LED2" gate="G$1" x="403.86" y="142.24"/>
+<instance part="HL2" gate="G$1" x="370.84" y="198.12" rot="R90"/>
+<instance part="HL1" gate="G$1" x="403.86" y="142.24" smashed="yes">
+<attribute name="NAME" x="406.908" y="141.224" size="1.778" layer="95"/>
+<attribute name="VALUE" x="406.908" y="139.065" size="1.778" layer="96"/>
+</instance>
 <instance part="R25" gate="G$1" x="403.86" y="129.54" smashed="yes" rot="MR90">
 <attribute name="NAME" x="405.13" y="133.1214" size="1.778" layer="95" rot="MR180"/>
@@
 <pinref part="GND15" gate="1" pin="GND"/>
 <wire x1="254" y1="231.14" x2="254" y2="223.52" width="0.1524" layer="91"/>
+<pinref part="X3" gate="G$1" pin="7"/>
+<wire x1="256.54" y1="241.3" x2="254" y2="241.3" width="0.1524" layer="91"/>
+<wire x1="254" y1="241.3" x2="254" y2="231.14" width="0.1524" layer="91"/>
+<junction x="254" y="231.14"/>
 </segment>
 <segment>
@@
 <wire x1="335.28" y1="200.66" x2="335.28" y2="198.12" width="0.1524" layer="91"/>
 <junction x="335.28" y="198.12"/>
-<pinref part="LED1" gate="G$1" pin="A"/>
+<pinref part="HL2" gate="G$1" pin="A"/>
 <wire x1="365.76" y1="198.12" x2="368.3" y2="198.12" width="0.1524" layer="91"/>
 <junction x="365.76" y="198.12"/>
@@
 <junction x="378.46" y="147.32"/>
 <wire x1="396.24" y1="147.32" x2="403.86" y2="147.32" width="0.1524" layer="91"/>
-<pinref part="LED2" gate="G$1" pin="A"/>
+<pinref part="HL1" gate="G$1" pin="A"/>
 <wire x1="403.86" y1="147.32" x2="403.86" y2="144.78" width="0.1524" layer="91"/>
 <junction x="396.24" y="147.32"/>
@@
 <net name="N$39" class="0">
 <segment>
-<pinref part="LED2" gate="G$1" pin="C"/>
+<pinref part="HL1" gate="G$1" pin="C"/>
 <pinref part="R25" gate="G$1" pin="2"/>
 <wire x1="403.86" y1="137.16" x2="403.86" y2="134.62" width="0.1524" layer="91"/>
@@
 <net name="N$41" class="0">
 <segment>
-<pinref part="LED1" gate="G$1" pin="C"/>
+<pinref part="HL2" gate="G$1" pin="C"/>
 <pinref part="R26" gate="G$1" pin="2"/>
 <wire x1="375.92" y1="198.12" x2="378.46" y2="198.12" width="0.1524" layer="91"/>

Commit message: .
Parts:
- removed R1: (no value), rcl:R-EU_M1206
- added CP1: 100n, rcl:C-EUC0805
- added CP2: 220mf, Speccy:CPOL-EUE2.5-5
- added J1: (no value), rcl:R-EU_M1206
- C3Y: value 0.1 -> 100n
- X4: value (none) -> SD Card
- renumbered R1223 to R27
Connections:
- new net D2.: DD10A.A8, DD3G$1.I/O4, DD8.D2, J1.2
- net +5V: now also CP1.1, CP2.+
- net D2: now also J1.1; no longer DD10A.A8, DD3G$1.I/O4, DD8.D2
- net GND: now also CP1.2, CP2.-
Other:
- note added: "C DA1"
- note added: "C DD1"
- note added: "C DD12"
- note added: "C DD2"
- note added: "C DD3 DD10"
- note added: "C DD7"
- note added: "C DD8"
- moved on the sheet: R23

Commit message: .
Parts:
- added X3P: (no value), con-lstb:MA04-1
- R23: device rcl:R-EU_R0805 -> rcl:R-EU_R1206
Connections:
- removed net N$24: R2.2, R22.1, X3.1
- new net KDATR: R2.2, R22.1, X3.1, X3P.2
- net +5V: now also X3P.3
- net GND: now also X3P.4
- net KCLK: now also X3P.1
Changed lines of the file:
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@@
 <part name="R21" library="Speccy" deviceset="R-EU_" device="0207/10" value="10k"/>
 <part name="R22" library="rcl" deviceset="R-EU_" device="R0805" value="4k7"/>
-<part name="R23" library="rcl" deviceset="R-EU_" device="R0805" value="4k7"/>
+<part name="R23" library="rcl" deviceset="R-EU_" device="R1206" value="4k7"/>
 <part name="R1Y" library="rcl" deviceset="R-EU_" device="R0805" value="1k"/>
 <part name="GND7" library="supply1" deviceset="GND" device=""/>
@@
 <part name="CP2" library="Speccy" deviceset="CPOL-EU" device="E2.5-5" value="220mf"/>
 <part name="CP1" library="rcl" deviceset="C-EU" device="C0805" value="100n"/>
+<part name="X3P" library="con-lstb" deviceset="MA04-1" device=""/>
+<part name="P+17" library="supply1" deviceset="+5V" device=""/>
+<part name="GND29" library="supply1" deviceset="GND" device=""/>
 </parts>
 <sheets>
@@
 <instance part="CP2" gate="G$1" x="121.92" y="231.14"/>
 <instance part="CP1" gate="G$1" x="111.76" y="231.14"/>
+<instance part="X3P" gate="1" x="297.18" y="233.68" rot="MR0"/>
+<instance part="P+17" gate="1" x="284.48" y="241.3" smashed="yes">
+<attribute name="VALUE" x="287.02" y="243.84" size="1.778" layer="96" rot="R180"/>
+</instance>
+<instance part="GND29" gate="1" x="297.18" y="246.38" rot="MR0"/>
 </instances>
 <busses>
@@
 <wire x1="403.86" y1="124.46" x2="403.86" y2="121.92" width="0.1524" layer="91"/>
 </segment>
+<segment>
+<pinref part="X3P" gate="1" pin="4"/>
+<wire x1="289.56" y1="236.22" x2="289.56" y2="248.92" width="0.1524" layer="91"/>
+<pinref part="GND29" gate="1" pin="GND"/>
+<wire x1="289.56" y1="248.92" x2="297.18" y2="248.92" width="0.1524" layer="91"/>
+</segment>
 </net>
 <net name="+5V" class="0">
@@
 <wire x1="30.48" y1="228.6" x2="30.48" y2="231.14" width="0.1524" layer="91"/>
 </segment>
+<segment>
+<pinref part="P+17" gate="1" pin="+5V"/>
+<pinref part="X3P" gate="1" pin="3"/>
+<wire x1="289.56" y1="233.68" x2="284.48" y2="233.68" width="0.1524" layer="91"/>
+<wire x1="284.48" y1="233.68" x2="284.48" y2="238.76" width="0.1524" layer="91"/>
+</segment>
 </net>
 <net name="A0" class="0">
@@
 <label x="248.92" y="236.22" size="1.778" layer="95"/>
 </segment>
+<segment>
+<label x="279.4" y="228.6" size="1.778" layer="95"/>
+<wire x1="289.56" y1="228.6" x2="279.4" y2="228.6" width="0.1524" layer="91"/>
+<pinref part="X3P" gate="1" pin="1"/>
+</segment>
 </net>
 <net name="KDAT" class="0">
@@
 </segment>
 </net>
-<net name="N$24" class="0">
+<net name="KDATR" class="0">
 <segment>
 <pinref part="R2" gate="G$1" pin="2"/>
@@
 <wire x1="241.3" y1="228.6" x2="241.3" y2="226.06" width="0.1524" layer="91"/>
 <junction x="241.3" y="226.06"/>
+<label x="243.84" y="226.06" size="1.778" layer="95"/>
+</segment>
+<segment>
+<label x="279.4" y="231.14" size="1.778" layer="95"/>
+<wire x1="289.56" y1="231.14" x2="279.4" y2="231.14" width="0.1524" layer="91"/>
+<pinref part="X3P" gate="1" pin="2"/>
 </segment>
 </net>

Commit message: .
Parts:
- R2: device rcl:R-EU_M1206 -> rcl:R-EU_R1206
Other:
- moved on the sheet: X3P
Changed lines of the file:
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@@
 <part name="R9P2" library="rcl" deviceset="R-EU_" device="R1206" value="75"/>
 <part name="J1" library="rcl" deviceset="R-EU_" device="M1206"/>
-<part name="R2" library="rcl" deviceset="R-EU_" device="M1206"/>
+<part name="R2" library="rcl" deviceset="R-EU_" device="R1206"/>
 <part name="DD12" library="Speccy" deviceset="74*74" device="O" technology="LS" value="74LS74O"/>
 <part name="P+15" library="supply1" deviceset="+5V" device=""/>
@@
 <instance part="CP2" gate="G$1" x="121.92" y="231.14"/>
 <instance part="CP1" gate="G$1" x="111.76" y="231.14"/>
-<instance part="X3P" gate="1" x="297.18" y="233.68" rot="MR0"/>
-<instance part="P+17" gate="1" x="284.48" y="241.3" smashed="yes">
-<attribute name="VALUE" x="287.02" y="243.84" size="1.778" layer="96" rot="R180"/>
+<instance part="X3P" gate="1" x="276.86" y="233.68" smashed="yes" rot="MR180">
+<attribute name="VALUE" x="275.59" y="243.84" size="1.778" layer="96" rot="MR180"/>
+<attribute name="NAME" x="280.67" y="242.062" size="1.778" layer="95" rot="MR0"/>
 </instance>
-<instance part="GND29" gate="1" x="297.18" y="246.38" rot="MR0"/>
+<instance part="P+17" gate="1" x="287.02" y="243.84" smashed="yes">
+<attribute name="VALUE" x="289.56" y="246.38" size="1.778" layer="96" rot="R180"/>
+</instance>
+<instance part="GND29" gate="1" x="287.02" y="226.06" rot="MR0"/>
 </instances>
 <busses>
@@
 <segment>
 <pinref part="X3P" gate="1" pin="4"/>
-<wire x1="289.56" y1="236.22" x2="289.56" y2="248.92" width="0.1524" layer="91"/>
 <pinref part="GND29" gate="1" pin="GND"/>
-<wire x1="289.56" y1="248.92" x2="297.18" y2="248.92" width="0.1524" layer="91"/>
+<wire x1="284.48" y1="231.14" x2="287.02" y2="231.14" width="0.1524" layer="91"/>
+<wire x1="287.02" y1="231.14" x2="287.02" y2="228.6" width="0.1524" layer="91"/>
 </segment>
 </net>
@@
 <pinref part="P+17" gate="1" pin="+5V"/>
 <pinref part="X3P" gate="1" pin="3"/>
-<wire x1="289.56" y1="233.68" x2="284.48" y2="233.68" width="0.1524" layer="91"/>
-<wire x1="284.48" y1="233.68" x2="284.48" y2="238.76" width="0.1524" layer="91"/>
+<wire x1="284.48" y1="233.68" x2="287.02" y2="233.68" width="0.1524" layer="91"/>
+<wire x1="287.02" y1="233.68" x2="287.02" y2="241.3" width="0.1524" layer="91"/>
 </segment>
 </net>
@@
 </segment>
 <segment>
-<label x="279.4" y="228.6" size="1.778" layer="95"/>
-<wire x1="289.56" y1="228.6" x2="279.4" y2="228.6" width="0.1524" layer="91"/>
+<label x="289.56" y="238.76" size="1.778" layer="95"/>
+<wire x1="284.48" y1="238.76" x2="294.64" y2="238.76" width="0.1524" layer="91"/>
 <pinref part="X3P" gate="1" pin="1"/>
 </segment>
@@
 </segment>
 <segment>
-<label x="279.4" y="231.14" size="1.778" layer="95"/>
-<wire x1="289.56" y1="231.14" x2="279.4" y2="231.14" width="0.1524" layer="91"/>
+<label x="289.56" y="236.22" size="1.778" layer="95"/>
+<wire x1="284.48" y1="236.22" x2="294.64" y2="236.22" width="0.1524" layer="91"/>
 <pinref part="X3P" gate="1" pin="2"/>
 </segment>

Commit message: .
Parts:
- added CE2, CX1: 100n, rcl:C-EUC0805
Connections:
- net +5V: now also CE2.1, CX1.1
- net GND: now also CE2.2, CX1.2
Other:
- note added: "C DD9"
- note added: "C X1"
- moved on the sheet: CE1, CM16, CP1, CP2, CRL, CT, CW29, CY, CZ80, R2, R22, X3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

Commit message: .
Parts:
- CRL: device rcl:C-EUC1206 -> rcl:C-EUC0805
Changed lines of the file:
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@@
 <grid distance="100" unitdist="mil" unit="mil" style="lines" multiple="1" display="yes" altdistance="0.01" altunitdist="inch" altunit="inch"/>
 <layers>
-<layer number="1" name="Top" color="4" fill="1" visible="no" active="no"/>
-<layer number="2" name="Route2" color="1" fill="3" visible="no" active="no"/>
-<layer number="3" name="Route3" color="4" fill="3" visible="no" active="no"/>
-<layer number="4" name="Route4" color="1" fill="4" visible="no" active="no"/>
-<layer number="5" name="Route5" color="4" fill="4" visible="no" active="no"/>
-<layer number="6" name="Route6" color="1" fill="8" visible="no" active="no"/>
-<layer number="7" name="Route7" color="4" fill="8" visible="no" active="no"/>
-<layer number="8" name="Route8" color="1" fill="2" visible="no" active="no"/>
-<layer number="9" name="Route9" color="4" fill="2" visible="no" active="no"/>
-<layer number="10" name="Route10" color="1" fill="7" visible="no" active="no"/>
-<layer number="11" name="Route11" color="4" fill="7" visible="no" active="no"/>
-<layer number="12" name="Route12" color="1" fill="5" visible="no" active="no"/>
-<layer number="13" name="Route13" color="4" fill="5" visible="no" active="no"/>
-<layer number="14" name="Route14" color="1" fill="6" visible="no" active="no"/>
-<layer number="15" name="Route15" color="4" fill="6" visible="no" active="no"/>
-<layer number="16" name="Bottom" color="1" fill="1" visible="no" active="no"/>
-<layer number="17" name="Pads" color="2" fill="1" visible="no" active="no"/>
-<layer number="18" name="Vias" color="2" fill="1" visible="no" active="no"/>
-<layer number="19" name="Unrouted" color="6" fill="1" visible="no" active="no"/>
-<layer number="20" name="Dimension" color="15" fill="1" visible="no" active="no"/>
-<layer number="21" name="tPlace" color="7" fill="1" visible="no" active="no"/>
-<layer number="22" name="bPlace" color="7" fill="1" visible="no" active="no"/>
-<layer number="23" name="tOrigins" color="15" fill="1" visible="no" active="no"/>
-<layer number="24" name="bOrigins" color="15" fill="1" visible="no" active="no"/>
-<layer number="25" name="tNames" color="7" fill="1" visible="no" active="no"/>
-<layer number="26" name="bNames" color="7" fill="1" visible="no" active="no"/>
-<layer number="27" name="tValues" color="7" fill="1" visible="no" active="no"/>
-<layer number="28" name="bValues" color="7" fill="1" visible="no" active="no"/>
+<layer number="1" name="Top" color="4" fill="1" visible="yes" active="no"/>
+<layer number="2" name="Route2" color="1" fill="3" visible="yes" active="no"/>
+<layer number="3" name="Route3" color="4" fill="3" visible="yes" active="no"/>
+<layer number="4" name="Route4" color="1" fill="4" visible="yes" active="no"/>
+<layer number="5" name="Route5" color="4" fill="4" visible="yes" active="no"/>
+<layer number="6" name="Route6" color="1" fill="8" visible="yes" active="no"/>
+<layer number="7" name="Route7" color="4" fill="8" visible="yes" active="no"/>
+<layer number="8" name="Route8" color="1" fill="2" visible="yes" active="no"/>
+<layer number="9" name="Route9" color="4" fill="2" visible="yes" active="no"/>
+<layer number="10" name="Route10" color="1" fill="7" visible="yes" active="no"/>
+<layer number="11" name="Route11" color="4" fill="7" visible="yes" active="no"/>
+<layer number="12" name="Route12" color="1" fill="5" visible="yes" active="no"/>
+<layer number="13" name="Route13" color="4" fill="5" visible="yes" active="no"/>
+<layer number="14" name="Route14" color="1" fill="6" visible="yes" active="no"/>
+<layer number="15" name="Route15" color="4" fill="6" visible="yes" active="no"/>
+<layer number="16" name="Bottom" color="1" fill="1" visible="yes" active="no"/>
+<layer number="17" name="Pads" color="2" fill="1" visible="yes" active="no"/>
+<layer number="18" name="Vias" color="2" fill="1" visible="yes" active="no"/>
+<layer number="19" name="Unrouted" color="6" fill="1" visible="yes" active="no"/>
+<layer number="20" name="Dimension" color="15" fill="1" visible="yes" active="no"/>
+<layer number="21" name="tPlace" color="7" fill="1" visible="yes" active="no"/>
+<layer number="22" name="bPlace" color="7" fill="1" visible="yes" active="no"/>
+<layer number="23" name="tOrigins" color="15" fill="1" visible="yes" active="no"/>
+<layer number="24" name="bOrigins" color="15" fill="1" visible="yes" active="no"/>
+<layer number="25" name="tNames" color="7" fill="1" visible="yes" active="no"/>
+<layer number="26" name="bNames" color="7" fill="1" visible="yes" active="no"/>
+<layer number="27" name="tValues" color="7" fill="1" visible="yes" active="no"/>
+<layer number="28" name="bValues" color="7" fill="1" visible="yes" active="no"/>
 <layer number="29" name="tStop" color="7" fill="3" visible="no" active="no"/>
 <layer number="30" name="bStop" color="7" fill="6" visible="no" active="no"/>
@@
 <layer number="35" name="tGlue" color="7" fill="4" visible="no" active="no"/>
 <layer number="36" name="bGlue" color="7" fill="5" visible="no" active="no"/>
-<layer number="37" name="tTest" color="7" fill="1" visible="no" active="no"/>
-<layer number="38" name="bTest" color="7" fill="1" visible="no" active="no"/>
+<layer number="37" name="tTest" color="7" fill="1" visible="yes" active="no"/>
+<layer number="38" name="bTest" color="7" fill="1" visible="yes" active="no"/>
 <layer number="39" name="tKeepout" color="4" fill="11" visible="no" active="no"/>
 <layer number="40" name="bKeepout" color="1" fill="11" visible="no" active="no"/>
@@
 <layer number="44" name="Drills" color="7" fill="1" visible="no" active="no"/>
 <layer number="45" name="Holes" color="7" fill="1" visible="no" active="no"/>
-<layer number="46" name="Milling" color="3" fill="1" visible="no" active="no"/>
-<layer number="47" name="Measures" color="7" fill="1" visible="no" active="no"/>
-<layer number="48" name="Document" color="7" fill="1" visible="no" active="no"/>
-<layer number="49" name="Reference" color="7" fill="1" visible="no" active="no"/>
-<layer number="50" name="dxf" color="7" fill="1" visible="no" active="no"/>
-<layer number="51" name="tDocu" color="7" fill="1" visible="no" active="no"/>
-<layer number="52" name="bDocu" color="7" fill="1" visible="no" active="no"/>
-<layer number="53" name="tGND_GNDA" color="7" fill="9" visible="no" active="no"/>
-<layer number="54" name="bGND_GNDA" color="1" fill="9" visible="no" active="no"/>
-<layer number="56" name="wert" color="7" fill="1" visible="no" active="no"/>
-<layer number="57" name="tCAD" color="7" fill="1" visible="no" active="no"/>
+<layer number="46" name="Milling" color="3" fill="1" visible="yes" active="no"/>
+<layer number="47" name="Measures" color="7" fill="1" visible="yes" active="no"/>
+<layer number="48" name="Document" color="7" fill="1" visible="yes" active="no"/>
+<layer number="49" name="Reference" color="7" fill="1" visible="yes" active="no"/>
+<layer number="50" name="dxf" color="7" fill="1" visible="yes" active="no"/>
+<layer number="51" name="tDocu" color="7" fill="1" visible="yes" active="no"/>
+<layer number="52" name="bDocu" color="7" fill="1" visible="yes" active="no"/>
+<layer number="53" name="tGND_GNDA" color="7" fill="9" visible="yes" active="no"/>
+<layer number="54" name="bGND_GNDA" color="1" fill="9" visible="yes" active="no"/>
+<layer number="56" name="wert" color="7" fill="1" visible="yes" active="no"/>
+<layer number="57" name="tCAD" color="7" fill="1" visible="yes" active="no"/>
 <layer number="90" name="Modules" color="5" fill="1" visible="yes" active="yes"/>
 <layer number="91" name="Nets" color="2" fill="1" visible="yes" active="yes"/>
@@
 <part name="CZ80" library="rcl" deviceset="C-EU" device="C0805" value="100n"/>
 <part name="CW29" library="rcl" deviceset="C-EU" device="C1206" value="100n"/>
-<part name="CRL" library="rcl" deviceset="C-EU" device="C1206" value="100n"/>
+<part name="CRL" library="rcl" deviceset="C-EU" device="C0805" value="100n"/>
 <part name="GND20" library="supply1" deviceset="GND" device=""/>
 <part name="VT1" library="transistor" deviceset="*-NPN-" device="TO92-CBE" technology="BC550" value="BC337(KT503)"/>
@@
 <text x="63.5" y="238.76" size="1.778" layer="91">C
 DD2</text>
-<text x="144.78" y="238.76" size="1.778" layer="91">C
+<text x="142.24" y="238.76" size="1.778" layer="91">C
 X1</text>
 </plain>

Commit message: .
Parts:
- R19: device rcl:R-EU_M1206 -> rcl:R-EU_M0805
Changed lines of the file:
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@@
 <part name="GND6" library="supply1" deviceset="GND" device=""/>
 <part name="R24" library="Speccy" deviceset="R-EU_" device="0207/10" value="2k2"/>
-<part name="R19" library="rcl" deviceset="R-EU_" device="M1206" value="10k"/>
+<part name="R19" library="rcl" deviceset="R-EU_" device="M0805" value="10k"/>
 <part name="R20" library="rcl" deviceset="R-EU_" device="R0805" value="10k"/>
 <part name="R21" library="Speccy" deviceset="R-EU_" device="0207/10" value="10k"/>

Commit message: .
Parts:
- R26: device rcl:R-EU_R0805 -> rcl:R-EU_R1206
Changed lines of the file:
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@@
 <part name="R25" library="rcl" deviceset="R-EU_" device="R0805" value="1k"/>
 <part name="GND27" library="supply1" deviceset="GND" device=""/>
-<part name="R26" library="rcl" deviceset="R-EU_" device="R0805" value="1k"/>
+<part name="R26" library="rcl" deviceset="R-EU_" device="R1206" value="1k"/>
 <part name="CP2" library="Speccy" deviceset="CPOL-EU" device="E2.5-5" value="220mf"/>
 <part name="CP1" library="rcl" deviceset="C-EU" device="C0805" value="100n"/>
