File: Speccy2007_128KY.brd (EAGLE design)
At the start: 168.6 x 112.4 mm, 119 parts, among them J1 0, J2 0, J3 0, X1 5V, X2 SCART-F, X3 PS/2 KB, X3P KB, X4 SD Card, X5 ByteBlaster, X6 AVRISP

Commit message: .
Parts:
- added C7P*: 33, rcl:C1206
- R43: device rcl:R1206 -> rcl:R0805
- moved C6P 1.27 mm to (24.1, 64.6)
- moved Z2 0.95 mm to (34.0, 64.1)
- moved R6P 0.63 mm to (23.5, 62.1)
- renumbered R5P to R5P*
Connections:
- new net N$63: C7P*.1, DA1.17
- net GND: now also C7P*.2
Routing:
- net N$63: track 0.00 -> 3.05 mm
- net FCI: track 48.1 -> 46.3 mm
- net N$45: track 33.8 -> 34.6 mm
- net N$52: track 8.82 -> 8.19 mm
- net N$53: track 3.49 -> 2.86 mm
- net GND: track 1252.9 -> 1253.5 mm
- net N$7: track 23.3 -> 22.7 mm

Commit message: ..
Parts:
- DD11: value К555ЛН1 -> 74LS04
- DD12: value К155ТМ2 -> 74LS74
- DD9: device ref-pack_:DIL40 -> Speccy:DIL40
- J3: value 0 -> (none); device rcl:R0805 -> jumper:SJ
- VT1: value KT503Г(BC337) -> BC337
- moved C2P 9.94 mm to (6.99, 17.6)
- moved C3P 9.94 mm to (16.5, 14.8)
- renumbered C20P to C12P, C8P1 to C10P, C8P2 to C11P, R9P1 to R10P, R9P2 to R11P
Connections:
- net N$13: now also C2P.1; no longer C3P.1
- net N$14: now also C3P.1; no longer C2P.1
- net N$35: now also C3P.2; no longer C2P.2
- net N$46: now also C2P.2; no longer C3P.2
