File: Speccy2007_128KY.brd (EAGLE design)
At the start: 168.6 x 112.4 mm, 120 parts, among them J1 0, J2 0, X1 5V, X2 SCART-F, X3 PS/2 KB, X3P KB, X4 SD Card, X5 ByteBlaster, X6 AVRISP

Commit message: power
Parts:
- moved R43 0.32 mm to (73.0, 79.9)
Routing:
- net +5V: track 886.9 -> 907.2 mm
Changed lines of the file:
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@@
 <setting verticaltext="up"/>
 </settings>
-<grid distance="6.25" unitdist="mil" unit="mil" style="lines" multiple="1" display="yes" altdistance="0.025" altunitdist="inch" altunit="inch"/>
+<grid distance="12.5" unitdist="mil" unit="mil" style="lines" multiple="1" display="yes" altdistance="0.025" altunitdist="inch" altunit="inch"/>
 <layers>
 <layer number="1" name="Top" color="4" fill="1" visible="yes" active="yes"/>
@@
 <wire x1="40.9575" y1="46.19625" x2="41.5925" y2="46.83125" width="0.1524" layer="21"/>
 <wire x1="41.5925" y1="46.83125" x2="42.8625" y2="46.83125" width="0.1524" layer="21"/>
+<rectangle x1="17.62125" y1="26.67" x2="19.84375" y2="28.8925" layer="16"/>
+<rectangle x1="13.81125" y1="26.67" x2="16.03375" y2="28.8925" layer="16"/>
+<rectangle x1="10.00125" y1="26.67" x2="12.22375" y2="28.8925" layer="16"/>
+<rectangle x1="13.81125" y1="22.86" x2="16.03375" y2="25.0825" layer="16"/>
+<rectangle x1="17.62125" y1="22.86" x2="19.84375" y2="25.0825" layer="16"/>
+<rectangle x1="10.00125" y1="22.86" x2="12.22375" y2="25.0825" layer="16"/>
+<rectangle x1="17.62125" y1="19.05" x2="19.84375" y2="21.2725" layer="16"/>
+<rectangle x1="13.81125" y1="19.05" x2="16.03375" y2="21.2725" layer="16"/>
 </plain>
 <attributes>
@@
 <attribute name="VALUE" x="72.7075" y="96.04375" size="1.27" layer="28" rot="MR270"/>
 </element>
-<element name="R43" library="rcl" package="R0805" value="2k" x="73.025" y="79.53375" smashed="yes" rot="MR270">
-<attribute name="NAME" x="75.08875" y="69.5325" size="1.27" layer="26" rot="MR0"/>
-<attribute name="VALUE" x="74.77125" y="67.945" size="1.27" layer="28" rot="MR0"/>
+<element name="R43" library="rcl" package="R0805" value="2k" x="73.025" y="79.85125" smashed="yes" rot="MR270">
+<attribute name="NAME" x="75.08875" y="69.85" size="1.27" layer="26" rot="MR0"/>
+<attribute name="VALUE" x="74.77125" y="68.2625" size="1.27" layer="28" rot="MR0"/>
 </element>
 <element name="R44" library="rcl" package="R1206" value="1k" x="70.8025" y="76.99375" smashed="yes" rot="MR90">
@@
 <wire x1="64.135" y1="77.62625" x2="61.9125" y2="77.62625" width="0.8128" layer="16"/>
 <wire x1="64.135" y1="77.62625" x2="66.3575" y2="77.62625" width="0.8128" layer="16"/>
-<wire x1="51.7525" y1="77.62625" x2="46.6725" y2="77.62625" width="0.8128" layer="16"/>
-<wire x1="46.6725" y1="77.62625" x2="39.0525" y2="77.62625" width="0.8128" layer="16"/>
-<wire x1="39.0525" y1="77.62625" x2="39.0525" y2="72.86625" width="0.8128" layer="16"/>
-<wire x1="46.6725" y1="72.86625" x2="46.6725" y2="77.62625" width="0.8128" layer="16"/>
 <contactref element="C13" pad="1"/>
-<wire x1="39.0525" y1="77.62625" x2="33.9725" y2="77.62625" width="0.8128" layer="16"/>
 <wire x1="138.1125" y1="10.31875" x2="140.0175" y2="10.31875" width="0.8128" layer="16"/>
 <wire x1="140.0175" y1="10.31875" x2="141.2875" y2="9.04875" width="0.8128" layer="16"/>
@@
 <wire x1="116.04625" y1="84.29625" x2="118.58625" y2="81.43875" width="0.4064" layer="16"/>
 <wire x1="120.97" y1="81.75625" x2="118.58625" y2="81.43875" width="0.4064" layer="16"/>
-<wire x1="72.39" y1="76.99375" x2="73.66" y2="76.04125" width="0.4064" layer="16"/>
-<wire x1="73.66" y1="76.04125" x2="77.47" y2="76.04125" width="0.8128" layer="16"/>
-<wire x1="77.47" y1="78.26625" x2="77.47" y2="76.04125" width="0.8128" layer="16"/>
-<wire x1="77.47" y1="76.04125" x2="77.47" y2="73.18375" width="0.8128" layer="16"/>
-<wire x1="77.47" y1="73.18375" x2="77.1525" y2="72.86625" width="0.4064" layer="16"/>
 <wire x1="48.5775" y1="26.82875" x2="46.355" y2="28.73375" width="0.4064" layer="16"/>
 <wire x1="40.9575" y1="35.71875" x2="45.085" y2="30.63875" width="0.4064" layer="16"/>
@@
 <wire x1="15.5575" y1="76.99375" x2="15.5575" y2="71.12" width="0.3048" layer="16"/>
 <wire x1="16.1925" y1="70.32625" x2="15.5575" y2="71.12" width="0.4064" layer="16"/>
-<wire x1="74.6125" y1="42.5425" x2="74.295" y2="33.3375" width="0" layer="19" extent="16-16"/>
-<wire x1="40.9575" y1="43.33875" x2="52.07" y2="44.60875" width="0" layer="19" extent="16-16"/>
+<wire x1="38.735" y1="78.89625" x2="46.6725" y2="78.89625" width="2.54" layer="16"/>
+<wire x1="39.0525" y1="72.86625" x2="39.0525" y2="77.30875" width="1.27" layer="16"/>
+<wire x1="39.0525" y1="77.30875" x2="38.735" y2="78.89625" width="1.27" layer="16"/>
+<wire x1="46.6725" y1="72.86625" x2="46.6725" y2="78.89625" width="1.27" layer="16"/>
+<wire x1="38.735" y1="78.89625" x2="31.115" y2="78.89625" width="2.54" layer="16"/>
+<wire x1="48.255" y1="79.375" x2="66.3575" y2="79.375" width="2.54" layer="16"/>
+<wire x1="46.6725" y1="78.89625" x2="48.255" y2="79.375" width="2.54" layer="16"/>
+<wire x1="77.47" y1="78.26625" x2="77.47" y2="75.8825" width="1.27" layer="16"/>
+<wire x1="77.47" y1="75.8825" x2="77.47" y2="73.3425" width="1.27" layer="16"/>
+<wire x1="77.47" y1="73.3425" x2="77.1525" y2="72.86625" width="1.27" layer="16"/>
+<wire x1="73.81875" y1="75.8825" x2="77.47" y2="75.8825" width="1.27" layer="16"/>
+<wire x1="73.81875" y1="75.8825" x2="72.7075" y2="76.99375" width="0.8128" layer="16"/>
+<wire x1="72.7075" y1="76.99375" x2="72.39" y2="76.99375" width="0.8128" layer="16"/>
+<wire x1="80.01" y1="102.79125" x2="80.01" y2="102.87" width="0" layer="19" extent="1-16"/>
+<wire x1="52.07" y1="44.60875" x2="40.9575" y2="43.33875" width="0" layer="19" extent="16-16"/>
+<wire x1="74.295" y1="33.3375" x2="74.6125" y2="42.5425" width="0" layer="19" extent="16-16"/>
 </signal>
 <signal name="A0">
@@
 <wire x1="66.0375" y1="83.02625" x2="65.7225" y2="83.65875" width="0.3048" layer="16"/>
 <wire x1="65.7225" y1="83.65875" x2="65.7225" y2="89.69375" width="0.3048" layer="16"/>
-<wire x1="66.0375" y1="83.02625" x2="67.945" y2="82.07375" width="0.4064" layer="16"/>
-<wire x1="67.945" y1="82.07375" x2="67.945" y2="80.16875" width="0.4064" layer="16"/>
+<wire x1="66.0375" y1="83.02625" x2="68.2625" y2="81.75625" width="0.4064" layer="16"/>
 <wire x1="65.7225" y1="90.32875" x2="65.7225" y2="89.69375" width="0.4064" layer="16"/>
-<wire x1="67.945" y1="80.16875" x2="70.0155" y2="79.05075" width="0.4064" layer="16"/>
-<wire x1="70.0155" y1="79.05075" x2="70.8025" y2="78.41575" width="0.4064" layer="16"/>
-<wire x1="70.8025" y1="78.41575" x2="73.025" y2="78.58375" width="0.6096" layer="16"/>
-<wire x1="73.025" y1="78.58375" x2="75.2475" y2="78.26625" width="0.6096" layer="16"/>
+<wire x1="70.8025" y1="78.41575" x2="73.025" y2="78.90125" width="0.6096" layer="16"/>
+<wire x1="73.025" y1="78.90125" x2="75.2475" y2="78.26625" width="0.6096" layer="16"/>
 <wire x1="65.7225" y1="90.32875" x2="63.5" y2="92.55125" width="0.4064" layer="16"/>
 <wire x1="63.5" y1="92.55125" x2="63.1825" y2="92.55125" width="0.4064" layer="16"/>
+<wire x1="70.8025" y1="78.41575" x2="68.2625" y2="80.95575" width="0.4064" layer="16"/>
+<wire x1="68.2625" y1="80.95575" x2="68.2625" y2="81.75625" width="0.4064" layer="16"/>
 </signal>
 <signal name="SOUND_L">
@@
 <wire x1="75.8825" y1="82.70875" x2="74.93" y2="82.07375" width="0.4064" layer="16"/>
 <wire x1="74.93" y1="82.07375" x2="74.143" y2="82.07375" width="0.4064" layer="16"/>
-<wire x1="74.143" y1="82.07375" x2="73.025" y2="80.48375" width="0.4064" layer="16"/>
+<wire x1="74.143" y1="82.07375" x2="73.025" y2="80.80125" width="0.4064" layer="16"/>
 <wire x1="72.0725" y1="85.24625" x2="72.0725" y2="88.10625" width="0.4064" layer="16"/>
 <wire x1="72.3925" y1="85.56625" x2="72.0725" y2="85.24625" width="0.4064" layer="16"/>

Commit message: .
Routing:
- net +5V: track 907.2 -> 900.3 mm
- net N$64: track 0.00 -> 6.66 mm
- net N$7: track 22.4 -> 23.0 mm

Commit message: .
Routing:
- net +5V: track 900.3 -> 903.6 mm
- net GND: track 1253.5 -> 1254.8 mm
