File: Speccy2007_128KY.sch (EAGLE design)
At the start: 122 parts, among them J1 0, J2 0, J3 0, X1 5V, X2 SCART-F, X3 PS/2 KB, X3P KB, X4 SD Card, X5 ByteBlaster, X6 AVRISP

Commit message: clear
Parts:
- removed **R2: 2k2, rcl:R-EU_R1206
- removed *R1: 4k7, rcl:R-EU_R0805
- removed *R2: 2k2, rcl:R-EU_R0805
Connections:
- net GND: no longer **R2.1, *R2.1
- net SOUND_L: no longer *R1.1, *R2.2
- net SPEAKER: no longer **R2.2, *R1.2
Other:
- moved on the sheet: C1Y, C2Y, C3Y, R49

Commit message: .
Parts:
- added C7P*: 33, rcl:C-EUC1206
- R43: device rcl:R-EU_R1206 -> rcl:R-EU_R0805
- renumbered R5P to R5P*
Connections:
- new net N$63: C7P*.1, DA1.17
- net GND: now also C7P*.2
Other:
- moved on the sheet: C1, C10, C12, C13, C14, C15, C16, C17, C2, C3, C4, C5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

Commit message: .clear
Other:
- note added: "Speccy2007 128K Y PAL"
- note removed: "Speccy2007 128K Y"
- moved on the sheet: C1, C10, C12, C13, C14, C15, C16, C17, C1P, C1Y, C2, C20P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

Commit message: ..
Parts:
- removed R9P1, R9P2: 75, rcl:R-EU_R1206
- added R10P, R11P: 75, rcl:R-EU_R1206
- DD11: value К555ЛН1 -> 74LS04
- DD12: value К155ТМ2 -> 74LS74
- DD9: device ref-pack_:YM2149F -> Speccy:YM2149F
- J3: value 0 -> (none); device rcl:R-EU_R0805 -> jumper:SJ
- VT1: value KT503Г(BC337) -> BC337
- renumbered C20P to C12P, C8P1 to C10P, C8P2 to C11P
Connections:
- net B_OUT: now also R11P.1; no longer R9P2.1
- net G_OUT: now also R10P.1; no longer R9P1.1
- net N$13: now also C2P.1; no longer C3P.1
- net N$14: now also C3P.1; no longer C2P.1
- net N$34: now also R10P.2; no longer R9P1.2
- net N$35: now also C3P.2; no longer C2P.2
- net N$36: now also R11P.2; no longer R9P2.2
- net N$46: now also C2P.2; no longer C3P.2
- net RST_CPU: now also DD9.!RES; no longer DD9.-RES
Other:
- note added: "(AY-3-8910)"
- note added: "(UA880D)"
- note added: "JP1,JP2 default Video and RGB"
- note added: "KT503Г"
- note added: "PAL"
- note added: "RGB (R) --------------- S-Video(C)"
- note added: "Video -------------- S-Video(Y)"
- note added: "К155ТМ2"
- note added: "К555ЛН1"
- moved on the sheet: C1Y, C2P, C2Y, C3P, C3Y, DD2.10, DD2.11, DD2.12, DD2.13, DD2.14, DD2.15, DD2.16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

Commit message: ..
Other:
- note added: "R25-R32"
Changed lines of the file:
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@@
 ---------------
 S-Video(C)</text>
-<text x="370.84" y="109.22" size="1.778" layer="98">JP1,JP2 default
+<text x="355.6" y="60.96" size="1.778" layer="98">JP1,JP2 default
 Video and RGB</text>
 <text x="271.78" y="144.78" size="1.778" layer="98">(AY-3-8910)</text>
@@
 <text x="353.06" y="2.54" size="1.778" layer="98">К155ТМ2</text>
 <text x="30.48" y="132.08" size="1.778" layer="98">(UA880D)</text>
+<wire x1="361.315" y1="99.695" x2="361.315" y2="100.965" width="0.4064" layer="98"/>
+<wire x1="361.315" y1="84.455" x2="361.315" y2="85.725" width="0.4064" layer="98"/>
+<text x="302.26" y="154.94" size="1.778" layer="96">R25-R32</text>
 </plain>
 <instances>
@@
 <instance part="R25" gate="G$1" x="309.88" y="195.58" smashed="yes">
 <attribute name="NAME" x="308.61" y="197.0786" size="1.778" layer="95"/>
-<attribute name="VALUE" x="308.61" y="156.718" size="1.778" layer="96"/>
+<attribute name="VALUE" x="313.817" y="154.94" size="1.778" layer="96"/>
 </instance>
 <instance part="R26" gate="G$1" x="309.88" y="190.5" smashed="yes">
 <attribute name="NAME" x="308.61" y="191.9986" size="1.778" layer="95"/>
-<attribute name="VALUE" x="308.61" y="156.718" size="1.778" layer="96"/>
+<attribute name="VALUE" x="313.817" y="154.94" size="1.778" layer="96"/>
 </instance>
 <instance part="R27" gate="G$1" x="309.88" y="185.42" smashed="yes">
 <attribute name="NAME" x="308.61" y="186.9186" size="1.778" layer="95"/>
-<attribute name="VALUE" x="308.61" y="156.718" size="1.778" layer="96"/>
+<attribute name="VALUE" x="313.817" y="154.94" size="1.778" layer="96"/>
 </instance>
 <instance part="R28" gate="G$1" x="309.88" y="180.34" smashed="yes">
 <attribute name="NAME" x="308.61" y="181.8386" size="1.778" layer="95"/>
-<attribute name="VALUE" x="308.61" y="156.718" size="1.778" layer="96"/>
+<attribute name="VALUE" x="313.817" y="154.94" size="1.778" layer="96"/>
 </instance>
 <instance part="R29" gate="G$1" x="309.88" y="175.26" smashed="yes">
 <attribute name="NAME" x="308.61" y="176.7586" size="1.778" layer="95"/>
-<attribute name="VALUE" x="308.61" y="156.718" size="1.778" layer="96"/>
+<attribute name="VALUE" x="313.817" y="154.94" size="1.778" layer="96"/>
 </instance>
 <instance part="R30" gate="G$1" x="309.88" y="170.18" smashed="yes">
 <attribute name="NAME" x="308.61" y="171.6786" size="1.778" layer="95"/>
-<attribute name="VALUE" x="308.61" y="156.718" size="1.778" layer="96"/>
+<attribute name="VALUE" x="313.817" y="154.94" size="1.778" layer="96"/>
 </instance>
 <instance part="R31" gate="G$1" x="309.88" y="165.1" smashed="yes">
 <attribute name="NAME" x="308.61" y="166.5986" size="1.778" layer="95"/>
-<attribute name="VALUE" x="308.61" y="156.718" size="1.778" layer="96"/>
+<attribute name="VALUE" x="313.817" y="154.94" size="1.778" layer="96"/>
 </instance>
 <instance part="R32" gate="G$1" x="309.88" y="160.02" smashed="yes">
 <attribute name="NAME" x="308.61" y="161.5186" size="1.778" layer="95"/>
-<attribute name="VALUE" x="308.61" y="156.718" size="1.778" layer="96"/>
+<attribute name="VALUE" x="313.817" y="154.94" size="1.778" layer="96"/>
 </instance>
 <instance part="GND15" gate="1" x="238.76" y="215.9" rot="MR0"/>
@@
 <attribute name="VALUE" x="233.68" y="243.84" size="1.778" layer="96" rot="R180"/>
 </instance>
-<instance part="X2" gate="G$1" x="401.32" y="78.74"/>
+<instance part="X2" gate="G$1" x="401.32" y="78.74" smashed="yes">
+<attribute name="VALUE" x="396.24" y="48.26" size="1.778" layer="96"/>
+<attribute name="NAME" x="398.78" y="106.68" size="1.778" layer="95"/>
+</instance>
 <instance part="GND17" gate="1" x="411.48" y="48.26" rot="MR0"/>
 <instance part="GND18" gate="1" x="378.46" y="48.26" rot="MR0"/>
@@
 </instance>
 <instance part="R18" gate="G$1" x="325.12" y="165.1" smashed="yes" rot="R90">
-<attribute name="NAME" x="323.85" y="168.6814" size="1.778" layer="95" rot="R180"/>
-<attribute name="VALUE" x="323.85" y="165.862" size="1.778" layer="96" rot="R180"/>
+<attribute name="NAME" x="323.215" y="168.6814" size="1.778" layer="95" rot="R180"/>
+<attribute name="VALUE" x="323.215" y="165.862" size="1.778" layer="96" rot="R180"/>
 </instance>
 <instance part="R17" gate="G$1" x="325.12" y="180.34" smashed="yes" rot="R90">
-<attribute name="NAME" x="326.39" y="181.8386" size="1.778" layer="95"/>
-<attribute name="VALUE" x="326.39" y="177.038" size="1.778" layer="96"/>
+<attribute name="NAME" x="327.025" y="181.2036" size="1.778" layer="95"/>
+<attribute name="VALUE" x="327.025" y="178.308" size="1.778" layer="96"/>
 </instance>
 <instance part="R11" gate="G$1" x="355.6" y="187.96" smashed="yes" rot="R90">
 <attribute name="NAME" x="354.33" y="191.5414" size="1.778" layer="95" rot="R180"/>
-<attribute name="VALUE" x="354.33" y="188.722" size="1.778" layer="96" rot="R180"/>
+<attribute name="VALUE" x="353.695" y="188.722" size="1.778" layer="96" rot="R180"/>
 </instance>
 <instance part="R12" gate="G$1" x="347.98" y="165.1" smashed="yes" rot="R90">
 <attribute name="NAME" x="346.71" y="168.6814" size="1.778" layer="95" rot="R180"/>
-<attribute name="VALUE" x="346.71" y="165.862" size="1.778" layer="96" rot="R180"/>
+<attribute name="VALUE" x="346.075" y="165.862" size="1.778" layer="96" rot="R180"/>
 </instance>
 <instance part="R13" gate="G$1" x="347.98" y="187.96" smashed="yes" rot="R90">
 <attribute name="NAME" x="346.71" y="191.5414" size="1.778" layer="95" rot="R180"/>
-<attribute name="VALUE" x="346.71" y="188.722" size="1.778" layer="96" rot="R180"/>
+<attribute name="VALUE" x="346.075" y="188.722" size="1.778" layer="96" rot="R180"/>
 </instance>
 <instance part="R14" gate="G$1" x="340.36" y="165.1" smashed="yes" rot="R90">
-<attribute name="NAME" x="339.09" y="168.6814" size="1.778" layer="95" rot="R180"/>
-<attribute name="VALUE" x="339.09" y="165.862" size="1.778" layer="96" rot="R180"/>
+<attribute name="NAME" x="338.455" y="168.6814" size="1.778" layer="95" rot="R180"/>
+<attribute name="VALUE" x="338.455" y="165.862" size="1.778" layer="96" rot="R180"/>
 </instance>
 <instance part="R15" gate="G$1" x="340.36" y="187.96" smashed="yes" rot="R90">
 <attribute name="NAME" x="339.09" y="191.5414" size="1.778" layer="95" rot="R180"/>
-<attribute name="VALUE" x="339.09" y="188.722" size="1.778" layer="96" rot="R180"/>
+<attribute name="VALUE" x="338.455" y="188.722" size="1.778" layer="96" rot="R180"/>
 </instance>
 <instance part="R16" gate="G$1" x="332.74" y="187.96" smashed="yes" rot="R90">
-<attribute name="NAME" x="331.47" y="191.5414" size="1.778" layer="95" rot="R180"/>
-<attribute name="VALUE" x="331.47" y="188.722" size="1.778" layer="96" rot="R180"/>
+<attribute name="NAME" x="330.835" y="191.5414" size="1.778" layer="95" rot="R180"/>
+<attribute name="VALUE" x="330.835" y="188.722" size="1.778" layer="96" rot="R180"/>
 </instance>
 <instance part="GND21" gate="1" x="337.82" y="152.4" rot="MR0"/>
@@
 </instance>
 <instance part="R34" gate="G$1" x="401.32" y="127" smashed="yes" rot="MR90">
-<attribute name="NAME" x="402.59" y="130.5814" size="1.778" layer="95" rot="MR180"/>
-<attribute name="VALUE" x="402.59" y="127.762" size="1.778" layer="96" rot="MR180"/>
+<attribute name="NAME" x="407.67" y="128.4986" size="1.778" layer="95" rot="MR0"/>
+<attribute name="VALUE" x="407.67" y="126.238" size="1.778" layer="96" rot="MR0"/>
 </instance>
 <instance part="GND27" gate="1" x="401.32" y="116.84" rot="MR0"/>
